File: stm32-fpga-bootloader.kicad_sch (KiCad schematic)
At the start: 104 parts, among them J1 USB_C_Receptacle_USB2.0_14P, J10 Conn_02x16_Odd_Even, J2 JTAG, J7 USB_C_Receptacle_USB2.0_14P, J8 Conn_01x02, J9 Conn_01x02, SW1 RST, SW2 BOOT, SW3 RST, SW6 RST, U1 ACPL-798J-500E, U2 AMS1117-3.3, U3 RP2040, U4 W25Q128JVS, U5 LCMXO2-1200HC-4TG100I, U7 LMV321, U8 LMV321, Y1 12Mhz, Y3 ASE-xxxMHz

Commit message: Update the design files
Parts:
- removed C56, C57, C58, C59, C60, C61, C62, C63, C64, C65, C66, C67, C68, C69: 100n, Capacitor_SMD:C_0402_1005Metric, symbol Device:C_Small
- removed D10: SM4007, Diode_SMD:D_SOD-123F, symbol Diode:SM4007
- removed FB3, FB4, FB5, FB6: 600R@100Mhz, Inductor_SMD:L_0603_1608Metric, symbol Device:FerriteBead_Small
- removed R71, R72: 2.2k, Resistor_SMD:R_0402_1005Metric, symbol Device:R_Small
- removed U5: LCMXO2-1200HC-4TG100I, EasyEDA_Lib:TQFP-100_L14.0-W14.0-P0.50-LS16.0-TL, symbol EasyEDA_Lib:LCMXO2-1200HC-4TG100I
- removed Y3: ASE-xxxMHz, Oscillator:Oscillator_SMD_Abracon_ASE-4Pin_3.2x2.5mm_HandSoldering, symbol Oscillator:ASE-xxxMHz
- added J14: PMOD, Connector_PinSocket_2.54mm:PinSocket_2x06_P2.54mm_Horizontal, symbol Connector_Generic:Conn_02x06_Odd_Even
- added J15, J16, J17: Conn_01x12, Connector_PinHeader_1.27mm:PinHeader_1x12_P1.27mm_Vertical, symbol Connector_Generic:Conn_01x12
- H1, H2, H3, H4: footprint MountingHole:MountingHole_2.2mm_M2_ISO14580 -> MountingHole:MountingHole_2.7mm
Connections:
- net +3.3V: now also J14.11 (Pin_11), J14.12 (Pin_12)
- net GND: now also J14.10 (Pin_10), J14.9 (Pin_9)
- net displays/7SEG_D1: now also J15.1 (Pin_1)
- net displays/7SEG_D2: now also J15.2 (Pin_2)
- net displays/7SEG_D3: now also J15.3 (Pin_3)
- net displays/7SEG_D4: now also J15.4 (Pin_4)
- net displays/MATRIX_SPI_MOSI: now also J15.11 (Pin_11)
- net displays/MATRIX_SPI_SCK: now also J15.10 (Pin_10)
- net displays/MATRIX_SPI_nCS: now also J15.12 (Pin_12)
- net displays/SHIFT_REG_CLK: now also J15.5 (Pin_5)
- net displays/SHIFT_REG_DATA: now also J15.7 (Pin_7)
- net displays/SHIFT_REG_STCLK: now also J15.6 (Pin_6)
- net displays/SHIFT_REG_nMCLR: now also J15.8 (Pin_8)
- new net displays/SHIFT_REG_OE: J15.9 (Pin_9)
- no-connect marks 20 -> 19
Other:
- added sheet lcmxo2-cpld-block (lcmxo2-cpld-block.kicad_sch)
- sheet displays ports: added SHIFT_REG_OE; removed none
- moved on the sheet: C6, J10

Commit message: Update the schematic
Parts:
- removed C11, C12, C13: 10uF, Capacitor_SMD:C_0603_1608Metric, symbol Device:C_Small
- removed D6, D7: RED, LED_SMD:LED_0603_1608Metric, symbol Device:LED_Small
- removed H1, H2, H3, H4: MountingHole_Pad, MountingHole:MountingHole_2.7mm, symbol Mechanical:MountingHole_Pad
- removed J10: Conn_02x16_Odd_Even, Connector_PinSocket_1.27mm:PinSocket_2x16_P1.27mm_Vertical, symbol Connector_Generic:Conn_02x16_Odd_Even
- removed J2: JTAG, Connector_PinHeader_2.54mm:PinHeader_1x04_P2.54mm_Vertical, symbol Connector_Generic:Conn_01x04
- removed R17, R18: 1.2K, Resistor_SMD:R_0402_1005Metric, symbol Device:R_Small
- removed SW1, SW3, SW6: RST, Button_Switch_SMD:SW_SPST_TL3342, symbol Switch:SW_Push
- removed U2: AMS1117-3.3, Package_TO_SOT_SMD:SOT-223-3_TabPin2, symbol Regulator_Linear:AMS1117-3.3
- added A1: RaspberryPi_Pico, Module:RaspberryPi_Pico_Common_THT, symbol MCU_Module:RaspberryPi_Pico_Debug
- added H1, H2, H3, H4: MountingHole, MountingHole:MountingHole_3.2mm_M3, symbol Mechanical:MountingHole
- added J10: Jumpber, Connector_PinHeader_1.27mm:PinHeader_1x03_P1.27mm_Vertical, symbol Connector_Generic:Conn_01x03
- added J11, J9: Jumper, Connector_PinHeader_1.27mm:PinHeader_1x03_P1.27mm_Vertical, symbol Connector_Generic:Conn_01x03
- added J19: Conn_01x02, TerminalBlock_Phoenix:TerminalBlock_Phoenix_PT-1,5-2-3.5-H_1x02_P3.50mm_Horizontal, symbol Connector_Generic:Conn_01x02
- added R13: 10R, Resistor_SMD:R_0402_1005Metric, symbol Device:R_Small
- added R73, R74, R75, R76, R77, R78: 100R, Resistor_SMD:R_0402_1005Metric, symbol Device:R_Small
- added R82, R83, R84, R85, R86: 1.2K, Resistor_SMD:R_0603_1608Metric, symbol Device:R_Small
- added SW2: RUN, EasyEDA_Lib:SW-SMD_L3.9-W3.0-P4.45, symbol EasyEDA_Lib:TS-1088-AR02016
- added SW3: ICE_BTN, EasyEDA_Lib:SW-SMD_L3.9-W3.0-P4.45, symbol EasyEDA_Lib:TS-1088-AR02016
- added SW4: ICE_RST, EasyEDA_Lib:SW-SMD_L3.9-W3.0-P4.45, symbol EasyEDA_Lib:TS-1088-AR02016
- C1: renamed from C2; now not fitted; now left out of the parts list
- C10: renamed from C7; now not fitted; now left out of the parts list
- C2: renamed from C1; now not fitted; now left out of the parts list
- C3: renamed from C27; now not fitted; now left out of the parts list
- C4, J1, Y1: now not fitted; now left out of the parts list
- C5: renamed from C3; now not fitted; now left out of the parts list
- C6: renamed from C9; now not fitted; now left out of the parts list
- C7: renamed from C8; now not fitted; now left out of the parts list
- C8: renamed from C5; now not fitted; now left out of the parts list
- C9: renamed from C6; now not fitted; now left out of the parts list
- R1: renamed from R3; now not fitted; now left out of the parts list
- R2: renamed from R10; now not fitted; now left out of the parts list
- R3: renamed from R5; now not fitted; now left out of the parts list
- R4: renamed from R6; now not fitted; now left out of the parts list
- R5: renamed from R4; now not fitted; now left out of the parts list
- R6: renamed from R2; now not fitted; now left out of the parts list
- SW1: renamed from SW2; now not fitted; now left out of the parts list
- U1: renamed from U3; now not fitted; now left out of the parts list
- U2: renamed from U4; now not fitted; now left out of the parts list
- renumbered C30 to C11, C31 to C12, C28 to C13, C29 to C14, C47 to C15, C15 to C16, C44 to C17, C45 to C18, C46 to C19, D5 to D1, J9 to J2, J8 to J3, J7 to J4, J14 to J5, J17 to J6, J16 to J7, J15 to J8, R1 to R10, R29 to R11, R30 to R12, R31 to R14, R14 to R15, R15 to R16, R32 to R17, R33 to R18, R22 to R19, R23 to R20, R24 to R21, R25 to R22, R26 to R23, R27 to R24, R19 to R25, R20 to R26, R21 to R27, R43 to R28, R42 to R29, R41 to R30, R44 to R31, R16 to R7, R28 to R8, R13 to R9, U8 to U3, U7 to U4, U1 to U5
Connections:
- net ENCODER_A: now also J10.1 (Pin_1)
- net ENCODER_B: now also J10.2 (Pin_2)
- net ENCODER_BTN: now also J10.3 (Pin_3)
- net GND: now also A1.13 (GND), A1.18 (GND), A1.23 (GND), A1.28 (GND), A1.3 (GND), A1.33 (AGND), A1.38 (GND), A1.8 (GND), A1.D2 (GND), J19.2 (Pin_2), R84.1, R86.1, SW2.1, SW3.1, SW4.1
- net ICE_BTN: now also SW3.2
- net ICE_CDONE: now also A1.21 (GPIO16)
- net ICE_SPI_MISO: now also A1.16 (GPIO12)
- net ICE_SPI_MOSI: now also A1.15 (GPIO11)
- net ICE_SPI_SCK: now also A1.19 (GPIO14), R13.2
- net ICE_SPI_SS: now also A1.17 (GPIO13)
- net ICE_nRST: now also A1.20 (GPIO15), SW4.2
- net RPI_ICE0: now also A1.1 (GPIO0)
- net RPI_ICE1: now also A1.2 (GPIO1)
- net RPI_ICE2: now also A1.4 (GPIO2)
- net RPI_ICE3: now also A1.5 (GPIO3)
- net RPI_ICE4: now also A1.6 (GPIO4)
- net RPI_ICE5: now also A1.7 (GPIO5)
- net RPI_ICE6: now also A1.9 (GPIO6)
- net RPI_ICE7: now also A1.10 (GPIO7)
- net UART1_RX: now also A1.12 (GPIO9)
- net UART1_TX: now also A1.11 (GPIO8)
- net at R10.2: now also A1.30 (RUN), SW2.2; no longer U1.26 (RUN)
- net IOB_0a: now reaches J5.1 (Pin_1)
- net IOB_5b: now reaches J5.2 (Pin_2)
- net IOB_2a: now reaches J5.3 (Pin_3)
- net IOB_6a: now reaches J5.4 (Pin_4)
- net IOB_3b_G6: now reaches J5.5 (Pin_5)
- net IOB_8a: now reaches J5.6 (Pin_6)
- net IOB_4a: now reaches J5.7 (Pin_7)
- net IOT_51a: now reaches J5.8 (Pin_8)
- net at U5.10 (MDAT-): now also R73.1, R75.2
- net at U5.11 (MDAT+): now also R73.2, R74.2
- net at U5.12 (MCLKIN−): now also R76.1, R78.2
- net at U5.13 (MCLKIN+): now also R76.2, R77.2
- net at U5.2 (VIN+): now also R85.2
- net at U5.3 (VIN-): now also R86.2
- new net: R83.2, R84.2, R85.1
- new net: J19.1 (Pin_1), R82.1
- new net: A1.14 (GPIO10), R13.1
- new net: R82.2, R83.1
- no-connect marks 19 -> 22
Other:
- note removed: "JTAG"
- note removed: "LDO"
- moved on the sheet: C15, C16, C17, C18, C19, J4, J5, R10, R25, R26, R27, R28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

Commit message: Update the schematic
Parts:
- added R87: 10k, Resistor_SMD:R_0402_1005Metric, symbol Device:R_Small
Connections:
- net +3.3V: now also R87.1
- net ICE_BTN: now also R87.2
- net ICE_SPI_SCK: no longer R13.2
- net IOB_13b: now also J6.4 (Pin_4)
- net IOB_16a: now also J6.8 (Pin_8)
- net IOB_18a: now also J6.2 (Pin_2)
- net IOB_20a: now also J6.6 (Pin_6)
- net IOB_22a: now also J6.3 (Pin_3)
- net IOB_23b: now also J6.7 (Pin_7)
- net IOT_37a: now also J6.5 (Pin_5)
- net IOT_50b: now also J6.1 (Pin_1)
- net PB18C: now reaches R74.1
- net PB18B: now reaches R78.1
- net PB18D: now reaches R75.1
- net PB15A: now reaches J11.1 (Pin_1)
- net PB15B: now reaches J11.2 (Pin_2)
- net PB11B/PCLKC2_1: now reaches J11.3 (Pin_3)
- net PB18A: now reaches R77.1
- net IOT_44b: now reaches J6.10 (Pin_10)
- net IOT_39a: now reaches J6.11 (Pin_11)
- net IOT_48b: now reaches J6.12 (Pin_12)
- net IOT_43a: now reaches J6.9 (Pin_9)
- net CPLD_B0_PT10A: now reaches A1.22 (GPIO17)
- net CPLD_B1_PT10B: now reaches A1.24 (GPIO18)
- net CPLD_B2_PT9A: now reaches A1.25 (GPIO19)
- net CPLD_B3_PT9B: now reaches A1.26 (GPIO20)
- net CPLD_B4_PR9A: now reaches A1.27 (GPIO21)
- net CPLD_B5_PR9B: now reaches A1.29 (GPIO22)
- net CPLD_B6_PR9C: now reaches A1.32 (GPIO27_ADC1)
- net CPLD_B7_PR9D: now reaches A1.34 (GPIO28_ADC2)
- net IOT_38b: now reaches J9.1 (Pin_1)
- net IOT_36b: now reaches J9.2 (Pin_2)
- net IOT_45a_G1: now reaches J9.3 (Pin_3)
- new net ICE_CLOCK: R13.2
Other:
- sheet lcmxo2-cpld-block ports: added CPLDK_SCK, CPLD_B0_PT10A, CPLD_B1_PT10B, CPLD_B2_PT9A, CPLD_B3_PT9B, CPLD_B4_PR9A, CPLD_B5_PR9B, CPLD_B6_PR9C, CPLD_B7_PR9D, CPLD_MISO, CPLD_MOSI, CPLD_SCL, CPLD_SDA, CPLD_SPI_CS, CPLD_SPI_MCS, PB11B/PCLKC2_1, PB15A, PB15B, PB18A, PB18B, PB18C, PB18D, PT10C/TDO, PT10D/TDI, PT11C/TCK, PT11D/TMS, PT15C/JTAGENB, PT15D/PROGRAMN, PT17D/DONE; removed none
- moved on the sheet: C15, C16, C17, C18, C19, J10, J11, J19, J6, J7, J8, J9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

Commit message: update the  source code
Parts:
- added J21, J22: Conn_02x05_Top_Bottom, Connector_PinHeader_2.54mm:PinHeader_2x05_P2.54mm_Vertical, symbol Connector_Generic:Conn_02x05_Top_Bottom
Connections:
- net +3.3V: now also J22.10 (Pin_10)
- net CPLD_B0_PT10A: no longer A1.22 (GPIO17)
- net CPLD_B1_PT10B: no longer A1.24 (GPIO18)
- net CPLD_B2_PT9A: no longer A1.25 (GPIO19)
- net CPLD_B3_PT9B: no longer A1.26 (GPIO20)
- net CPLD_B4_PR9A: no longer A1.27 (GPIO21)
- net CPLD_B5_PR9B: no longer A1.29 (GPIO22)
- net CPLD_B6_PR9C: no longer A1.32 (GPIO27_ADC1)
- net CPLD_B7_PR9D: no longer A1.34 (GPIO28_ADC2)
- net GND: now also J22.5 (Pin_5)
- net ICE_CDONE: now also A1.29 (GPIO22); no longer A1.21 (GPIO16)
- net GPIO26_ADC0: now reaches A1.31 (GPIO26_ADC0)
- net GPIO26_ADC0: now also J22.8 (Pin_8)
- new net GPIO16_SPI0_RX: A1.21 (GPIO16), J22.3 (Pin_3)
- new net GPIO17_SPI0_CSn: A1.22 (GPIO17), J22.4 (Pin_4)
- new net GPIO18_SPI0_SCK: A1.24 (GPIO18), J22.1 (Pin_1)
- new net GPIO19_SPI0_TX: A1.25 (GPIO19), J22.2 (Pin_2)
- new net GPIO20_I2C0_SDA: A1.26 (GPIO20), J22.6 (Pin_6)
- new net GPIO21_I2C0_SCL: A1.27 (GPIO21), J22.7 (Pin_7)
- new net GPIO27_ADC1: A1.32 (GPIO27_ADC1), J22.9 (Pin_9)
- no-connect marks 22 -> 24
Other:
- moved on the sheet: J7

Commit message: update the  source code
Parts:
- added J23, J24: CPLD-TO-RPI, Connector_PinHeader_2.54mm:PinHeader_2x05_P2.54mm_Vertical, symbol Connector_Generic:Conn_02x05_Top_Bottom
- J22: value Conn_02x05_Top_Bottom -> RPI-TO-CPLD
Connections:
- net +3.3V: now also J23.10 (Pin_10), J24.10 (Pin_10)
- net CPLD_B0_PT10A: now also J24.9 (Pin_9)
- net CPLD_B1_PT10B: now also J24.8 (Pin_8)
- net CPLD_B2_PT9A: now also J24.7 (Pin_7)
- net CPLD_B3_PT9B: now also J24.6 (Pin_6)
- net CPLD_B4_PR9A: now also J24.1 (Pin_1)
- net CPLD_B5_PR9B: now also J24.2 (Pin_2)
- net CPLD_B6_PR9C: now also J24.3 (Pin_3)
- net CPLD_B7_PR9D: now also J24.4 (Pin_4)
- net GND: now also J23.5 (Pin_5), J24.5 (Pin_5)
- net GPIO16_SPI0_RX: now also J23.3 (Pin_3)
- net GPIO17_SPI0_CSn: now also J23.4 (Pin_4)
- net GPIO18_SPI0_SCK: now also J23.1 (Pin_1)
- net GPIO19_SPI0_TX: now also J23.2 (Pin_2)
- net GPIO20_I2C0_SDA: now also J23.6 (Pin_6)
- net GPIO21_I2C0_SCL: now also J23.7 (Pin_7)
- net GPIO26_ADC0: now also J23.8 (Pin_8)
- net GPIO27_ADC1: now also J23.9 (Pin_9)
Other:
- sheet lcmxo2-cpld-block ports: added PL5A/PCLKT3_1; removed none

Commit message: update the  source code
Parts:
- removed C11, C12: 100n, Capacitor_SMD:C_0402_1005Metric, symbol Device:C_Small
- removed J10: Jumpber, Connector_PinHeader_1.27mm:PinHeader_1x03_P1.27mm_Vertical, symbol Connector_Generic:Conn_01x03
- removed J11, J9: Jumper, Connector_PinHeader_1.27mm:PinHeader_1x03_P1.27mm_Vertical, symbol Connector_Generic:Conn_01x03
- removed J2: Conn_01x02, TerminalBlock_Phoenix:TerminalBlock_Phoenix_PT-1,5-2-3.5-H_1x02_P3.50mm_Horizontal, symbol Connector_Generic:Conn_01x02
- removed J21: Conn_02x05_Top_Bottom, Connector_PinHeader_2.54mm:PinHeader_2x05_P2.54mm_Vertical, symbol Connector_Generic:Conn_02x05_Top_Bottom
- removed J22: RPI-TO-CPLD, Connector_PinHeader_2.54mm:PinHeader_2x05_P2.54mm_Vertical, symbol Connector_Generic:Conn_02x05_Top_Bottom
- removed J23, J24: CPLD-TO-RPI, Connector_PinHeader_2.54mm:PinHeader_2x05_P2.54mm_Vertical, symbol Connector_Generic:Conn_02x05_Top_Bottom
- removed J6, J7, J8: Conn_01x12, Connector_PinHeader_1.27mm:PinHeader_1x12_P1.27mm_Vertical, symbol Connector_Generic:Conn_01x12
- removed R11, R12, R14, R17, R18: 1.2K, Resistor_SMD:R_0402_1005Metric, symbol Device:R_Small
- removed R8: 1R, Resistor_SMD:R_0402_1005Metric, symbol Device:R_Small
- removed U3: LMV321, Package_TO_SOT_SMD:SOT-23-5, symbol Amplifier_Operational:LMV321
- added J2: TO-LCD, KiCadLocal:CON_536470274_MOL, symbol Connector_Generic:Conn_02x11_Odd_Even
- added J22: RPI-TO-CPLD, Connector_PinHeader_2.54mm:PinHeader_2x06_P2.54mm_Vertical, symbol Connector_Generic:Conn_02x06_Top_Bottom
- added J23, J24: CPLD-TO-RPI, Connector_PinHeader_2.54mm:PinHeader_2x06_P2.54mm_Vertical, symbol Connector_Generic:Conn_02x06_Top_Bottom
- added JP1, JP2, JP3, JP4, JP5, JP6: Jumper, Connector_PinHeader_2.54mm:PinHeader_1x03_P2.54mm_Vertical, symbol Jumper:Jumper_3_Bridged12
Connections:
- net +3.3V: now also J22.12 (Pin_12), J23.12 (Pin_12), J24.12 (Pin_12)
- net CPLDK_SCK: now also J23.1 (Pin_1)
- net CPLD_B0_PT10A: now also J24.10 (Pin_10)
- net CPLD_B1_PT10B: now also J24.9 (Pin_9)
- net CPLD_B2_PT9A: now also J24.8 (Pin_8)
- net CPLD_B3_PT9B: now also J24.7 (Pin_7)
- net CPLD_B4_PR9A: now also J24.1 (Pin_1)
- net CPLD_B5_PR9B: now also J24.2 (Pin_2)
- net CPLD_B6_PR9C: now also J24.3 (Pin_3)
- net CPLD_B7_PR9D: now also J24.4 (Pin_4)
- net CPLD_CLOCK: now also J23.10 (Pin_10), J23.5 (Pin_5), J24.5 (Pin_5)
- net CPLD_MISO: now also J23.3 (Pin_3)
- net CPLD_MOSI: now also J23.2 (Pin_2)
- net CPLD_SCL: now also J23.8 (Pin_8)
- net CPLD_SDA: now also J23.7 (Pin_7)
- net CPLD_SPI_CS: now also J23.4 (Pin_4)
- net CPLD_SPI_MCS: now also J23.9 (Pin_9)
- net ENCODER_A: now also JP4.2 (C)
- net ENCODER_B: now also JP5.2 (C)
- net ENCODER_BTN: now also JP6.2 (C)
- net GND: now also J2.11 (Pin_11), J2.12 (Pin_12), J22.6 (Pin_6), J23.6 (Pin_6), J24.6 (Pin_6)
- net GPIO16_SPI0_RX: now also J22.3 (Pin_3)
- net GPIO17_SPI0_CSn: now also J22.4 (Pin_4)
- net GPIO18_SPI0_SCK: now also J22.1 (Pin_1)
- net GPIO19_SPI0_TX: now also J22.2 (Pin_2)
- net GPIO20_I2C0_SDA: now also J22.7 (Pin_7)
- net GPIO21_I2C0_SCL: now also J22.8 (Pin_8)
- net GPIO26_ADC0: now also J22.9 (Pin_9)
- net GPIO27_ADC1: now also J22.10 (Pin_10)
- net ICE_CLOCK: now also J22.5 (Pin_5)
- net IOT_36b: now also JP5.1 (A)
- net IOT_38b: now also JP4.1 (A)
- net IOT_39a: now also JP2.1 (A)
- net IOT_44b: now also JP3.1 (A)
- net IOT_45a_G1: now also JP6.1 (A)
- net IOT_48b: now also JP1.1 (A)
- net PB11B/PCLKC2_1: now also JP6.3 (B)
- net PB15A: now also JP4.3 (B)
- net PB15B: now also JP5.3 (B)
- new net +5V: J2.7 (Pin_7), J2.8 (Pin_8)
- new net CLOCK: J2.17 (Pin_17)
- new net DIG_1: J2.1 (Pin_1)
- new net DIG_2: J2.2 (Pin_2)
- new net DIG_3: J2.4 (Pin_4)
- new net DIG_4: J2.6 (Pin_6)
- new net DIG_DP: J2.3 (Pin_3)
- new net IO: J2.16 (Pin_16)
- new net KEY: J2.18 (Pin_18)
- new net LED_SEG: J2.15 (Pin_15)
- new net MATRIX_SPI_MOSI: JP2.2 (C)
- new net MATRIX_SPI_SCK: JP1.2 (C)
- new net MATRIX_SPI_nCS: JP3.2 (C)
- new net PR10C: JP3.3 (B)
- new net PR10D: JP1.3 (B)
- new net PR8D: JP2.3 (B)
- new net RTSW_A: J2.19 (Pin_19)
- new net RTSW_B: J2.20 (Pin_20)
- no-connect marks 24 -> 59
Other:
- sheet displays ports: added none; removed 7SEG_D1, 7SEG_D2, 7SEG_D3, 7SEG_D4, SHIFT_REG_CLK, SHIFT_REG_DATA, SHIFT_REG_OE, SHIFT_REG_STCLK, SHIFT_REG_nMCLR
- sheet lcmxo2-cpld-block ports: added PB11A/PCLKT2_1, PB11C, PB11D, PB9A/PCLKT2_0, PB9B/PCLKC2_0, PL4A, PL4B, PR10C, PR10D, PR8A, PR8C, PR8D; removed none
- note added: "GPIO16_SPI0_RX GPIO19_SPI0_TX GPIO18_SPI0_SCK GPIO17_SPI0_CSn"
- moved on the sheet: C17, C18, C19, J4, J5, R25, R26, R27, R28, R29, R30, R31

Commit message: update the  source code
Connections:
- net ICE_X2 is gone; now on net IOB_20a: R25.2
Changed lines of the file:
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@@
 	(rectangle
 		(start 137.16 69.85)
-		(end 208.28 129.54)
+		(end 228.6 129.54)
 		(stroke
 			(width 0)
@@
 	(wire
 		(pts
-			(xy 245.11 58.42) (xy 264.16 58.42)
+			(xy 434.34 45.72) (xy 450.85 45.72)
 		)
 		(stroke
@@
 	(wire
 		(pts
-			(xy 434.34 45.72) (xy 450.85 45.72)
+			(xy 240.03 58.42) (xy 264.16 58.42)
 		)
 		(stroke
@@
 		)
 	)
+	(label "ICE_USB_P"
+		(at 245.11 43.18 180)
+		(effects
+			(font
+				(size 1.27 1.27)
+			)
+			(justify right bottom)
+		)
+	)
 	(label "DIG_3"
 		(at 398.78 187.96 180)
@@
 		)
 	)
+	(label "IOB_20a"
+		(at 199.39 114.3 0)
+		(effects
+			(font
+				(size 1.27 1.27)
+			)
+			(justify left bottom)
+		)
+	)
 	(label "RPI_ICE2"
 		(at 245.11 66.04 0)
@@
 		)
 	)
-	(label "ICE_X2"
-		(at 199.39 114.3 180)
-		(effects
-			(font
-				(size 1.27 1.27)
-			)
-			(justify right bottom)
-		)
-	)
 	(label "RPI_ICE3"
 		(at -166.37 88.9 180)
@@
 		(effects
 			(font
+				(size 1.27 1.27)
+			)
+			(justify right bottom)
+		)
+	)
+	(label "ICE_USB_N"
+		(at 240.03 58.42 180)
+		(effects
+			(font

Commit message: Update the source code
Parts:
- removed J4: USB_C_Receptacle_USB2.0_14P, Connector_USB:USB_C_Receptacle_G-Switch_GT-USB-7010ASV, symbol Connector:USB_C_Receptacle_USB2.0_14P
- added A2: RaspberryPi_Pico, Module:RaspberryPi_Pico_Common_THT, symbol MCU_Module:RaspberryPi_Pico_Debug
- added J4: USB FPGA, Connector_PinHeader_2.54mm:PinHeader_1x03_P2.54mm_Vertical, symbol Connector_Generic:Conn_01x03
- renumbered C13 to C11, C14 to C12, C17 to C13, C18 to C14, C19 to C17, J3 to J2, J22 to J3, J19 to J6, J2 to J7, J23 to J8, J24 to J9, JP3 to JP1, JP4 to JP2, JP2 to JP3, JP5 to JP4, JP1 to JP5, R13 to R10, R15 to R11, R16 to R12, R19 to R13, R20 to R14, R21 to R15, R22 to R16, R23 to R17, R24 to R18, R87 to R19, R25 to R20, R26 to R21, R27 to R22, R82 to R23, R83 to R24, R84 to R25, R85 to R26, R86 to R27, R76 to R30, R73 to R31, R30 to R32, R77 to R33, R78 to R34, R74 to R35, R75 to R36, R31 to R37, R9 to R8, R10 to R9, U4 to U3, U5 to U4
Connections:
- net D+: no longer R20.1, R22.1
- net D-: no longer R21.1
- net GND: now also A2.13 (GND), A2.18 (GND), A2.23 (GND), A2.28 (GND), A2.3 (GND), A2.38 (GND), A2.8 (GND), A2.D2 (GND), J4.3 (Pin_3)
- new net: J4.1 (Pin_1), R21.1
- new net: J4.2 (Pin_2), R20.1, R22.1
- no-connect marks 59 -> 57
Other:
- removed sheet jtag-prog
- moved on the sheet: J3
