File: stm32-fpga-bootloader.kicad_pcb (KiCad board)
At the start: 2 copper layers, 100 x 65 mm, 176 parts, among them J1 USB_C_Receptacle_USB2.0_14P, J10 Conn_02x16_Odd_Even, J2 JTAG, J3 LEDX, J4 LEDY, J5 USB_C_Receptacle_USB2.0_14P, J6 Conn_ST_STDC14, J7 USB_C_Receptacle_USB2.0_14P, J8 Conn_01x02, J9 Conn_01x02, Q1 2N7002K, Q2 2N7002K, Q3 2N7002K, Q4 2N7002K, Q6 2N7002K, Q7 2N7002K, Q8 2N7002K, SW1 RST, SW2 BOOT, SW3 RST, SW6 RST, U1 ACPL-798J-500E, U10 W25Q128JVS, U11 74HC595D, U12 LTC-3743KD, U14 AMS1117-3.3, U15 MAX7221xNG, U16 FT2232HQ, U17 93LCxxA, U2 AMS1117-3.3, U3 RP2040, U4 W25Q128JVS, U6 LP5907MFX-1.2, U7 LMV321, U8 LMV321, U9 ICE40UP5K-SG48ITR, Y1 12Mhz, Y2 12Mhz

Commit message: Update the design files
Parts:
- added C57: 100n, Capacitor_SMD:C_0402_1005Metric, F.Cu at (168.8, 91.4)
- added C58: 100n, Capacitor_SMD:C_0402_1005Metric, F.Cu at (162.3, 92.2)
- added C59: 100n, Capacitor_SMD:C_0402_1005Metric, F.Cu at (158.6, 90.2)
- added C61: 100n, Capacitor_SMD:C_0402_1005Metric, F.Cu at (174.8, 97.4)
- added C62: 100n, Capacitor_SMD:C_0402_1005Metric, F.Cu at (174.8, 106.2)
- added C63: 100n, Capacitor_SMD:C_0402_1005Metric, F.Cu at (158.1, 119.2)
- added C64: 100n, Capacitor_SMD:C_0402_1005Metric, F.Cu at (155.1, 101.4)
- added C65: 100n, Capacitor_SMD:C_0402_1005Metric, F.Cu at (155.1, 98.4)
- added C66: 100n, Capacitor_SMD:C_0402_1005Metric, F.Cu at (154.8, 107.4)
- added C67: 100n, Capacitor_SMD:C_0402_1005Metric, F.Cu at (168.8, 112.6)
- added C68: 100n, Capacitor_SMD:C_0402_1005Metric, F.Cu at (158.8, 112.4)
- added D10: SM4007, Diode_SMD:D_SOD-123F, F.Cu at (155.8, 90.4)
- added FB3: 600R@100Mhz, Inductor_SMD:L_0603_1608Metric, F.Cu at (174.1, 92.2)
- added FB4: 600R@100Mhz, Inductor_SMD:L_0603_1608Metric, F.Cu at (174.3, 110.9)
- added FB5: 600R@100Mhz, Inductor_SMD:L_0603_1608Metric, F.Cu at (154.3, 95.7)
- added FB6: 600R@100Mhz, Inductor_SMD:L_0603_1608Metric, F.Cu at (156.6, 112.4)
- added J11: Raspberry_Pi_2_3, Connector_PinHeader_2.54mm:PinHeader_2x20_P2.54mm_Vertical, F.Cu at (134.2, 85.2)
- added J12: Conn_ST_STDC14, Connector_PinHeader_1.27mm:PinHeader_2x07_P1.27mm_Vertical, F.Cu at (148.7, 96.8)
- added J13: PMOD, Connector_PinSocket_2.54mm:PinSocket_2x06_P2.54mm_Horizontal, F.Cu at (144.7, 124.4)
- added J14: PMOD, Connector_PinSocket_2.54mm:PinSocket_2x06_P2.54mm_Horizontal, F.Cu at (162.3, 35.9)
- added J15: Conn_01x12, Connector_PinHeader_1.27mm:PinHeader_1x12_P1.27mm_Vertical, F.Cu at (176.6, 69.9)
- added J16: Conn_01x12, Connector_PinHeader_1.27mm:PinHeader_1x12_P1.27mm_Vertical, F.Cu at (176.6, 71.2)
- added J17: Conn_01x12, Connector_PinHeader_1.27mm:PinHeader_1x12_P1.27mm_Vertical, F.Cu at (176.6, 68.6)
- added R71: 2.2k, Resistor_SMD:R_0402_1005Metric, F.Cu at (166.3, 91.4)
- added R72: 2.2k, Resistor_SMD:R_0402_1005Metric, F.Cu at (167.6, 91.4)
- added Y3: ASE-xxxMHz, Oscillator:Oscillator_SMD_Abracon_ASE-4Pin_3.2x2.5mm_HandSoldering, F.Cu at (162.9, 120.3)
- C24: value 10uF -> 1uF
- H1, H2, H3, H4: footprint MountingHole:MountingHole_2.2mm_M2_ISO14580 -> MountingHole:MountingHole_2.7mm
- TP1: footprint Connector_Pin:Pin_D0.9mm_L10.0mm_W2.4mm_FlatFork -> Connector_Pin:Pin_D0.7mm_L6.5mm_W1.8mm_FlatFork
- U5: value ~ -> LCMXO2-1200HC-4TG100I; footprint EasyEDA_Lib:TQFP-100_L14.0-W14.0-P0.50-LS16.0-TL -> Package_QFP:TQFP-100_14x14mm_P0.5mm
- moved C14 155.9 mm to (252.7, 111.3)
- moved U12 153.7 mm to (198.6, 86.0)
- moved J6 134.6 mm to (138.2, 102.8), turned to -90 degrees
- moved U17 129.7 mm to (130.8, 126.2)
- moved U16 120.8 mm to (129.3, 114.5), turned to 180 degrees
- moved U1 120.8 mm to (188.8, 117.9)
- moved FB2 120.2 mm to (139.8, 117.2), turned to 180 degrees
- moved FB1 119.9 mm to (139.6, 114.2), turned to 180 degrees
- moved C49 118.3 mm to (136.6, 117.2), turned to 180 degrees
- moved C25 117.9 mm to (136.3, 114.2), turned to 180 degrees
- moved U15 117.8 mm to (201.9, 41.2)
- moved R61 114.8 mm to (138.3, 115.9)
- moved Q1 113.9 mm to (193.1, 94.7)
- moved R7 113.5 mm to (190.4, 105.5), turned to -90 degrees
- moved Q2 113.2 mm to (193.1, 98.3)
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Connections:
- net Net-(U11-OE#) renamed /displays/SHIFT_REG_OE
- U16 pad 1: unconnected-(U16-GND-Pad1) -> GND
- U16 pad 10: unconnected-(U16-AGND-Pad10) -> GND
- U16 pad 11: unconnected-(U16-GND-Pad11) -> GND
- U16 pad 15: unconnected-(U16-GND-Pad15) -> GND
- U16 pad 25: unconnected-(U16-GND-Pad25) -> GND
- U16 pad 35: unconnected-(U16-GND-Pad35) -> GND
- U16 pad 47: unconnected-(U16-GND-Pad47) -> GND
- U16 pad 5: unconnected-(U16-GND-Pad5) -> GND
- U16 pad 51: unconnected-(U16-GND-Pad51) -> GND
- U16 pad 65: unconnected-(U16-GND-Pad65) -> GND
- U5 pad 100: unconnected-(U5-VCC-Pad100) -> Net-(D10-K)
- U5 pad 20: unconnected-(U5-PL9A/PCLKT3_0-Pad20) -> /lcmxo2-cpld-block/PL9A/PCLKT3_0
- U5 pad 21: unconnected-(U5-PL9B/PCLKC3_0-Pad21) -> /lcmxo2-cpld-block/PL9B/PCLKC3_0
- U5 pad 24: unconnected-(U5-PL10C-Pad24) -> /lcmxo2-cpld-block/PL10C
- U5 pad 76: unconnected-(U5-PT17D/DONE-Pad76) -> /lcmxo2-cpld-block/PT17D/DONE
- U5 pad 77: unconnected-(U5-PT17C/INITN-Pad77) -> /lcmxo2-cpld-block/PT17C/INITN
- U5 pad 81: unconnected-(U5-PT15D/PROGRAMN-Pad81) -> /lcmxo2-cpld-block/PT15D/PROGRAMN
- U5 pad 82: unconnected-(U5-PT15C/JTAGENB-Pad82) -> /lcmxo2-cpld-block/PT15C/JTAGENB
- U5 pad 85: unconnected-(U5-PT12D/SDA/PCLKC0_0-Pad85) -> /lcmxo2-cpld-block/PT12D/SDA/PCLKC0_0
- U5 pad 86: unconnected-(U5-PT12C/SCL/PCLKT0_0-Pad86) -> /lcmxo2-cpld-block/PT12C/SCL/PCLKT0_0
- U5 pad 90: unconnected-(U5-PT11D/TMS-Pad90) -> /lcmxo2-cpld-block/PT11D/TMS
- U5 pad 91: unconnected-(U5-PT11C/TCK-Pad91) -> /lcmxo2-cpld-block/PT11C/TCK
- U5 pad 94: unconnected-(U5-PT10D/TDI-Pad94) -> /lcmxo2-cpld-block/PT10D/TDI
- U5 pad 95: unconnected-(U5-PT10C/TDO-Pad95) -> /lcmxo2-cpld-block/PT10C/TDO
Other:
- board size 100 x 65 mm -> 100 x 100 mm

Commit message: Update the schematic
Parts:
- removed C1, C3, C5, C8, C9: 100n, Capacitor_SMD:C_0402_1005Metric
- removed the C11 at (127.4, 52.2)
- removed the C12 at (116.6, 56.4)
- removed the C13 at (114.9, 56.5)
- removed C2, C4: 4.7u, Capacitor_SMD:C_0603_1608Metric
- removed the C27 at (152.7, 48.5)
- removed C6, C7: 10pF, Capacitor_SMD:C_0402_1005Metric
- removed J1: USB_C_Receptacle_USB2.0_14P, Connector_USB:USB_C_Receptacle_G-Switch_GT-USB-7010ASV
- removed the J2 at (161.3, 57.2)
- removed the R10 at (146.9, 57.4)
- removed R2: 1k, Resistor_SMD:R_0402_1005Metric
- removed R3: 240R, Resistor_SMD:R_0402_1005Metric
- removed R4: 10k, Resistor_SMD:R_0402_1005Metric
- removed R5, R6: 27R, Resistor_SMD:R_0402_1005Metric
- removed SW1, SW6: RST, Button_Switch_SMD:SW_SPST_TL3342
- removed U2: AMS1117-3.3, Package_TO_SOT_SMD:SOT-223-3_TabPin2
- removed the U3 at (145.8, 50.5)
- removed the U4 at (135.3, 55.0)
- removed Y1: 12Mhz, Crystal:Crystal_SMD_3225-4Pin_3.2x2.5mm
- added A1: RaspberryPi_Pico, Module:RaspberryPi_Pico_Common_THT, F.Cu at (116.2, 61.9)
- added D9: D_Schottky, Diode_SMD:D_SOD-123, F.Cu at (119.0, 106.4)
- added J11: Jumper, Connector_PinHeader_1.27mm:PinHeader_1x03_P1.27mm_Vertical, F.Cu at (181.9, 79.1)
- added J9: Jumper, Connector_PinHeader_1.27mm:PinHeader_1x03_P1.27mm_Vertical, F.Cu at (185.4, 79.1)
- added R13: 10R, Resistor_SMD:R_0402_1005Metric, F.Cu at (139.4, 59.1)
- added SW4: ICE_RST, EasyEDA_Lib:SW-SMD_L3.9-W3.0-P4.45, F.Cu at (129.9, 35.1)
- H1: renamed from H2; value MountingHole_Pad -> MountingHole; footprint MountingHole:MountingHole_2.7mm -> MountingHole:MountingHole_3.2mm_M3
- H2: renamed from H1; value MountingHole_Pad -> MountingHole; footprint MountingHole:MountingHole_2.7mm -> MountingHole:MountingHole_3.2mm_M3
- H3, H4: value MountingHole_Pad -> MountingHole; footprint MountingHole:MountingHole_2.7mm -> MountingHole:MountingHole_3.2mm_M3
- J10: value Conn_02x16_Odd_Even -> Jumpber; footprint Connector_PinSocket_1.27mm:PinSocket_2x16_P1.27mm_Vertical -> Connector_PinHeader_1.27mm:PinHeader_1x03_P1.27mm_Vertical
- SW2: value BOOT -> RUN; footprint Button_Switch_SMD:SW_SPST_TL3342 -> EasyEDA_Lib:SW-SMD_L3.9-W3.0-P4.45
- SW3: value RST -> ICE_BTN; footprint Button_Switch_SMD:SW_SPST_TL3342 -> EasyEDA_Lib:SW-SMD_L3.9-W3.0-P4.45
- U9: renamed from U11; footprint PCM_JLCPCB:SOIC-16_L9.9-W3.9-P1.27-LS6.0-BL -> PCM_JLCPCB:SOIC-16_3.9x9.9mm_P1.27mm
- moved J10 131.8 mm to (188.9, 79.1)
- moved SW3 103.6 mm to (134.4, 34.9), turned to 90 degrees
- moved C16 88.0 mm to (198.2, 109.9)
- moved D7 87.9 mm to (162.7, 32.7), turned to -90 degrees
- moved D6 85.4 mm to (165.7, 32.7), turned to -90 degrees
- moved R35 84.0 mm to (162.7, 36.1), turned to 90 degrees
- moved J17 81.9 mm to (208.9, 118.8), turned to 180 degrees
- moved R34 81.4 mm to (165.7, 36.2), turned to 90 degrees
- moved C35 71.3 mm to (197.2, 66.6)
- moved U10 61.5 mm to (137.6, 78.6), turned to 90 degrees
- moved U9 59.6 mm to (133.5, 73.4), turned to -90 degrees
- moved R40 59.5 mm to (127.4, 76.2), turned to 90 degrees
- moved Q3 58.0 mm to (143.2, 72.6)
- moved R45 58.0 mm to (140.5, 72.3)
- moved R46 58.0 mm to (145.9, 72.6)
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- renumbered C30 to C11, C31 to C12, C28 to C13, C29 to C14, C47 to C15, C15 to C16, C44 to C17, C45 to C18, C46 to C19, C32 to C20, C42 to C21, C33 to C22, C43 to C23, C35 to C24, C36 to C25, C34 to C26, C37 to C27, C19 to C28, C38 to C29, C39 to C30, C40 to C31, C20 to C32, C41 to C33, C10 to C34, C14 to C35, C18 to C36, C26 to C37, C21 to C38, C22 to C39, C16 to C40, C17 to C41, C48 to C42, C25 to C43, C49 to C44, C24 to C45, C23 to C46, C50 to C47, C54 to C48, C53 to C49, C52 to C50, C61 to C52, C57 to C53, C62 to C54, C58 to C55, C59 to C56, C67 to C57, C66 to C58, C68 to C59, C65 to C60, C64 to C61, C63 to C62, D5 to D1, D9 to D5, FB4 to FB3, FB3 to FB4, FB6 to FB5, FB5 to FB6, J3 to J12, J4 to J13, J5 to J14, J6 to J15, J13 to J16, J11 to J17, J12 to J18, J9 to J2, J8 to J3, J7 to J4, J14 to J5, J17 to J6, J16 to J7, J15 to J8, Q4 to Q1, Q1 to Q4, Q8 to Q5, R1 to R10, R29 to R11, R30 to R12, R31 to R14, R14 to R15, R15 to R16, R32 to R17, R33 to R18, R22 to R19, R23 to R20, R24 to R21, R25 to R22, R26 to R23, R27 to R24, R19 to R25, R20 to R26, R21 to R27, R43 to R28, R42 to R29, R41 to R30, R44 to R31, R36 to R32, R45 to R33, R17 to R34, R18 to R35, R37 to R36, R38 to R37, R39 to R38, R40 to R39, R47 to R40, R7 to R41, R58 to R42, R56 to R43, R9 to R44, R8 to R45, R57 to R46, R55 to R47, R11 to R48, R53 to R49, R49 to R50, R54 to R52, R50 to R53, R52 to R54, R46 to R55, R59 to R56, R35 to R57, R48 to R58, R60 to R59, R62 to R60, R63 to R62, R65 to R63, R66 to R65, R69 to R66, R70 to R67, R67 to R69, R16 to R7, R72 to R70, R28 to R8, R13 to R9, U12 to U10, U15 to U11, U17 to U12, U14 to U13, U16 to U14, U5 to U15, U8 to U3, U7 to U4, U1 to U5, U9 to U6, U10 to U7, U6 to U8
Connections:
- net /ICE_X1 renamed /IOT_50b
- net /ICE_X3 renamed /IOB_22a
- net /ICE_X4 renamed /IOB_13b
- net /ICE_X5 renamed /IOT_37a
- net /ICE_X6 renamed /IOB_20a
- net /ICE_X7 renamed /IOB_23b
- net /ICE_X8 renamed /IOB_16a
- J10 pad 1: unconnected-(J10-Pin_1-Pad1) -> /ENCODER_A
- J10 pad 2: unconnected-(J10-Pin_2-Pad2) -> /ENCODER_B
- J10 pad 3: unconnected-(J10-Pin_3-Pad3) -> /ENCODER_BTN
- J14 pad A4: VBUS -> Net-(D9-A)
- J14 pad A9: VBUS -> Net-(D9-A)
- J14 pad B4: VBUS -> Net-(D9-A)
- J14 pad B9: VBUS -> Net-(D9-A)
- J5 pad 1: unconnected-(J14-Pin_1-Pad1) -> /IOB_0a
- J5 pad 2: unconnected-(J14-Pin_2-Pad2) -> /IOB_5b
- J5 pad 3: unconnected-(J14-Pin_3-Pad3) -> /IOB_2a
- J5 pad 4: unconnected-(J14-Pin_4-Pad4) -> /IOB_6a
- J5 pad 5: unconnected-(J14-Pin_5-Pad5) -> /IOB_3b_G6
- J5 pad 6: unconnected-(J14-Pin_6-Pad6) -> /IOB_8a
- J5 pad 7: unconnected-(J14-Pin_7-Pad7) -> /IOB_4a
- J5 pad 8: unconnected-(J14-Pin_8-Pad8) -> /IOT_51a
- R10 pad 2: Net-(U3-RUN) -> Net-(A1-RUN)
- R34 pad 1: /ICE_LED1 -> /ice40-for-gpio/ICE_LED1
- R35 pad 1: /ICE_LED2 -> /ice40-for-gpio/ICE_LED2
- SW2 pad 1: /QSPI_SS -> GND
- SW2 pad 2: GND -> Net-(A1-RUN)
- U6 pad 10: /ICE_X2 -> /IOB_18a
- U6 pad 2: /ICE_Y6 -> /IOB_6a
- U6 pad 4: /ICE_Y7 -> /IOB_8a
- U6 pad 42: /ICE_Y8 -> /IOT_51a
- U6 pad 44: /ICE_Y3 -> /IOB_3b_G6
- U6 pad 45: /ICE_Y5 -> /IOB_5b
- U6 pad 46: /ICE_Y1 -> /IOB_0a
- U6 pad 47: /ICE_Y2 -> /IOB_2a
- U6 pad 48: /ICE_Y4 -> /IOB_4a

Commit message: update the  source code
Parts:
- removed C62: 100n, Capacitor_SMD:C_0402_1005Metric
- removed Y3: ASE-xxxMHz, Oscillator:Oscillator_SMD_Abracon_ASE-4Pin_3.2x2.5mm_HandSoldering
- added D11: RED, LED_SMD:LED_0603_1608Metric, F.Cu at (186.4, 124.0)
- added J19: Conn_01x02, TerminalBlock_Phoenix:TerminalBlock_Phoenix_PT-1,5-2-3.5-H_1x02_P3.50mm_Horizontal, F.Cu at (193.3, 127.0)
- added J20: Conn_02x04_Top_Bottom, Connector_PinHeader_2.54mm:PinHeader_2x04_P2.54mm_Vertical, F.Cu at (198.2, 71.2)
- added J21: Conn_02x04_Top_Bottom, Connector_PinHeader_2.54mm:PinHeader_2x04_P2.54mm_Vertical, F.Cu at (174.1, 78.8)
- added R72: 10k, Resistor_SMD:R_0402_1005Metric, F.Cu at (182.9, 123.7)
- added R73: 100R, Resistor_SMD:R_0402_1005Metric, F.Cu at (182.9, 107.8)
- added R74: 100R, Resistor_SMD:R_0402_1005Metric, F.Cu at (182.9, 109.8)
- added R75: 100R, Resistor_SMD:R_0402_1005Metric, F.Cu at (182.9, 111.8)
- added R76: 100R, Resistor_SMD:R_0402_1005Metric, F.Cu at (182.9, 113.8)
- added R77: 100R, Resistor_SMD:R_0402_1005Metric, F.Cu at (182.9, 115.8)
- added R78: 100R, Resistor_SMD:R_0402_1005Metric, F.Cu at (182.9, 117.8)
- added R79: 10k, Resistor_SMD:R_0402_1005Metric, F.Cu at (182.9, 125.7)
- added R80: 10k, Resistor_SMD:R_0402_1005Metric, F.Cu at (182.9, 127.7)
- added R81: 10k, Resistor_SMD:R_0402_1005Metric, F.Cu at (182.9, 129.7)
- added R82: 1.2K, Resistor_SMD:R_0603_1608Metric, F.Cu at (186.3, 108.1)
- added R83: 1.2K, Resistor_SMD:R_0603_1608Metric, F.Cu at (186.3, 110.6)
- added R84: 1.2K, Resistor_SMD:R_0603_1608Metric, F.Cu at (186.3, 113.1)
- added R85: 1.2K, Resistor_SMD:R_0603_1608Metric, F.Cu at (186.3, 115.6)
- added R86: 1.2K, Resistor_SMD:R_0603_1608Metric, F.Cu at (186.3, 118.1)
- added R87: 10k, Resistor_SMD:R_0402_1005Metric, F.Cu at (182.9, 119.8)
- moved C16 1.88 mm to (198.2, 108.0)
- moved U5 1.75 mm to (194.7, 115.9)
Connections:
- A1 pad 22: unconnected-(A1-GPIO17-Pad22) -> /CPLD_B0_PT10A
- A1 pad 24: unconnected-(A1-GPIO18-Pad24) -> /CPLD_B1_PT10B
- A1 pad 25: unconnected-(A1-GPIO19-Pad25) -> /CPLD_B2_PT9A
- A1 pad 26: unconnected-(A1-GPIO20-Pad26) -> /CPLD_B3_PT9B
- A1 pad 27: unconnected-(A1-GPIO21-Pad27) -> /CPLD_B4_PR9A
- A1 pad 29: unconnected-(A1-GPIO22-Pad29) -> /CPLD_B5_PR9B
- A1 pad 32: unconnected-(A1-GPIO27_ADC1-Pad32) -> /CPLD_B6_PR9C
- A1 pad 34: unconnected-(A1-GPIO28_ADC2-Pad34) -> /CPLD_B7_PR9D
- J11 pad 1: unconnected-(J11-Pin_1-Pad1) -> /PB15A
- J11 pad 2: unconnected-(J11-Pin_2-Pad2) -> /PB15B
- J11 pad 3: unconnected-(J11-Pin_3-Pad3) -> /PB11B/PCLKC2_1
- J16 pad 1: unconnected-(J16-Pin_1-Pad1) -> /lcmxo2-cpld-block/PL8A
- J16 pad 2: unconnected-(J16-Pin_2-Pad2) -> /lcmxo2-cpld-block/PL8B
- J16 pad 3: unconnected-(J16-Pin_3-Pad3) -> /lcmxo2-cpld-block/PL5D
- J16 pad 4: unconnected-(J16-Pin_4-Pad4) -> /lcmxo2-cpld-block/PL8D
- J16 pad 5: unconnected-(J16-Pin_5-Pad5) -> /lcmxo2-cpld-block/PL5C
- J16 pad 6: unconnected-(J16-Pin_6-Pad6) -> /lcmxo2-cpld-block/PL8C
- J16 pad 7: unconnected-(J16-Pin_7-Pad7) -> /lcmxo2-cpld-block/PL9B/PCLKC3_0
- J16 pad 8: unconnected-(J16-Pin_8-Pad8) -> /lcmxo2-cpld-block/PL9A/PCLKT3_0
- J17 pad 1: Net-(J17-3V3-Pad1) -> unconnected-(J17-3V3-Pad1)_1
- J17 pad 10: unconnected-(J17-GPIO15/RXD-Pad10) -> /lcmxo2-cpld-block/PB6B
- J17 pad 11: unconnected-(J17-GPIO17-Pad11) -> /lcmxo2-cpld-block/PR5D/PCLKC1_0
- J17 pad 12: unconnected-(J17-GPIO18/PWM0-Pad12) -> /lcmxo2-cpld-block/PR5C/PCLKT1_0
- J17 pad 13: unconnected-(J17-GPIO27-Pad13) -> /lcmxo2-cpld-block/PR2A
- J17 pad 14: Net-(J17-GND-Pad14) -> GND
- J17 pad 15: unconnected-(J17-GPIO22-Pad15) -> /lcmxo2-cpld-block/PR4B
- J17 pad 16: unconnected-(J17-GPIO23-Pad16) -> /lcmxo2-cpld-block/PR4A
- J17 pad 17: Net-(J17-3V3-Pad1) -> unconnected-(J17-3V3-Pad1)
- J17 pad 18: unconnected-(J17-GPIO24-Pad18) -> /lcmxo2-cpld-block/PR3B
- J17 pad 19: unconnected-(J17-MOSI0/GPIO10-Pad19) -> /lcmxo2-cpld-block/CPLD_MOSI
- J17 pad 2: Net-(J17-5V-Pad2) -> unconnected-(J17-5V-Pad2)
- J17 pad 20: Net-(J17-GND-Pad14) -> GND
- J17 pad 21: unconnected-(J17-MISO0/GPIO9-Pad21) -> /lcmxo2-cpld-block/CPLD_MISO
- J17 pad 22: unconnected-(J17-GPIO25-Pad22) -> /lcmxo2-cpld-block/PR3A
- J17 pad 23: unconnected-(J17-SCLK0/GPIO11-Pad23) -> /lcmxo2-cpld-block/CPLDK_SCK
- J17 pad 24: unconnected-(J17-~{CE0}/GPIO8-Pad24) -> /lcmxo2-cpld-block/CPLD_SPI_CS
- J17 pad 25: Net-(J17-GND-Pad14) -> GND
- J17 pad 26: unconnected-(J17-~{CE1}/GPIO7-Pad26) -> /lcmxo2-cpld-block/CPLD_SPI_MCS
- J17 pad 27: unconnected-(J17-ID_SD/GPIO0-Pad27) -> /lcmxo2-cpld-block/PB4D
- J17 pad 28: unconnected-(J17-ID_SC/GPIO1-Pad28) -> /lcmxo2-cpld-block/PT16C
- J17 pad 29: unconnected-(J17-GCLK1/GPIO5-Pad29) -> /lcmxo2-cpld-block/PT12A/PCLKT0_1
- J17 pad 3: unconnected-(J17-SDA/GPIO2-Pad3) -> /lcmxo2-cpld-block/CPLD_SDA
- J17 pad 30: Net-(J17-GND-Pad14) -> GND
- J17 pad 31: unconnected-(J17-GCLK2/GPIO6-Pad31) -> /lcmxo2-cpld-block/PT12B/PCLKC0_1
- J17 pad 32: unconnected-(J17-PWM0/GPIO12-Pad32) -> /lcmxo2-cpld-block/PT15A
- J17 pad 33: unconnected-(J17-PWM1/GPIO13-Pad33) -> /lcmxo2-cpld-block/PL3B/PCLKC3_2
- J17 pad 34: Net-(J17-GND-Pad14) -> GND
- J17 pad 35: unconnected-(J17-GPIO19/MISO1-Pad35) -> /lcmxo2-cpld-block/PR5A
- J17 pad 36: unconnected-(J17-GPIO16-Pad36) -> /lcmxo2-cpld-block/PR5B
- J17 pad 37: unconnected-(J17-GPIO26-Pad37) -> /lcmxo2-cpld-block/PR2B
- J17 pad 38: unconnected-(J17-GPIO20/MOSI1-Pad38) -> /lcmxo2-cpld-block/PR4D
- J17 pad 39: Net-(J17-GND-Pad14) -> GND
- J17 pad 4: Net-(J17-5V-Pad2) -> unconnected-(J17-5V-Pad2)_1
- J17 pad 40: unconnected-(J17-GPIO21/SCLK1-Pad40) -> /lcmxo2-cpld-block/PR4C
- J17 pad 5: unconnected-(J17-SCL/GPIO3-Pad5) -> /lcmxo2-cpld-block/CPLD_SCL
- J17 pad 6: Net-(J17-GND-Pad14) -> GND
- J17 pad 7: unconnected-(J17-GCLK0/GPIO4-Pad7) -> /lcmxo2-cpld-block/PT15B
- J17 pad 8: unconnected-(J17-GPIO14/TXD-Pad8) -> /lcmxo2-cpld-block/PB6A
- J17 pad 9: Net-(J17-GND-Pad14) -> GND
- J6 pad 1: unconnected-(J6-Pin_1-Pad1) -> /IOT_50b
- J6 pad 10: unconnected-(J6-Pin_10-Pad10) -> /IOT_44b
- J6 pad 11: unconnected-(J6-Pin_11-Pad11) -> /IOT_39a
- J6 pad 12: unconnected-(J6-Pin_12-Pad12) -> /IOT_48b
- J6 pad 2: unconnected-(J6-Pin_2-Pad2) -> /IOB_18a
- J6 pad 3: unconnected-(J6-Pin_3-Pad3) -> /IOB_22a
- J6 pad 4: unconnected-(J6-Pin_4-Pad4) -> /IOB_13b
- J6 pad 5: unconnected-(J6-Pin_5-Pad5) -> /IOT_37a
- J6 pad 6: unconnected-(J6-Pin_6-Pad6) -> /IOB_20a
- J6 pad 7: unconnected-(J6-Pin_7-Pad7) -> /IOB_23b
- J6 pad 8: unconnected-(J6-Pin_8-Pad8) -> /IOB_16a
- J6 pad 9: unconnected-(J6-Pin_9-Pad9) -> /IOT_43a
- J9 pad 1: unconnected-(J9-Pin_1-Pad1) -> /IOT_38b
- J9 pad 2: unconnected-(J9-Pin_2-Pad2) -> /IOT_36b
- J9 pad 3: unconnected-(J9-Pin_3-Pad3) -> /IOT_45a_G1
- R13 pad 2: /ICE_SPI_SCK -> /ICE_CLOCK
- R70 pad 1: /lcmxo2-cpld-block/PT12D/SDA/PCLKC0_0 -> /lcmxo2-cpld-block/CPLD_SDA
- R71 pad 1: /lcmxo2-cpld-block/PT12C/SCL/PCLKT0_0 -> /lcmxo2-cpld-block/CPLD_SCL
- U15 pad 13: unconnected-(U15-PL5B/PCLKC3_1-Pad13) -> /lcmxo2-cpld-block/PL5B/PCLKC3_1
- U15 pad 14: unconnected-(U15-PL5C-Pad14) -> /lcmxo2-cpld-block/PL5C
- U15 pad 15: unconnected-(U15-PL5D-Pad15) -> /lcmxo2-cpld-block/PL5D
- U15 pad 16: unconnected-(U15-PL8A-Pad16) -> /lcmxo2-cpld-block/PL8A
- U15 pad 17: unconnected-(U15-PL8B-Pad17) -> /lcmxo2-cpld-block/PL8B
- U15 pad 18: unconnected-(U15-PL8C-Pad18) -> /lcmxo2-cpld-block/PL8C
- U15 pad 19: unconnected-(U15-PL8D-Pad19) -> /lcmxo2-cpld-block/PL8D
- U15 pad 24: /lcmxo2-cpld-block/PL10C -> /lcmxo2-cpld-block/UART_TX
- U15 pad 25: unconnected-(U15-PL10D-Pad25) -> /lcmxo2-cpld-block/UART_RX
- U15 pad 27: unconnected-(U15-PB4C/CSSPIN-Pad27) -> /lcmxo2-cpld-block/CPLD_SPI_MCS
- U15 pad 28: unconnected-(U15-PB4D-Pad28) -> /lcmxo2-cpld-block/PB4D
- U15 pad 29: unconnected-(U15-PB6A-Pad29) -> /lcmxo2-cpld-block/PB6A
- U15 pad 30: unconnected-(U15-PB6B-Pad30) -> /lcmxo2-cpld-block/PB6B
- U15 pad 31: unconnected-(U15-PB6C/MCLK/CCLK-Pad31) -> /lcmxo2-cpld-block/CPLDK_SCK
- U15 pad 32: unconnected-(U15-PB6D/SO/SPISO-Pad32) -> /lcmxo2-cpld-block/CPLD_MISO
- U15 pad 39: unconnected-(U15-PB11B/PCLKC2_1-Pad39) -> /PB11B/PCLKC2_1
- U15 pad 4: unconnected-(U15-PL3B/PCLKC3_2-Pad4) -> /lcmxo2-cpld-block/PL3B/PCLKC3_2
- U15 pad 40: unconnected-(U15-PB15A-Pad40) -> /PB15A
- U15 pad 41: unconnected-(U15-PB15B-Pad41) -> /PB15B
- U15 pad 42: unconnected-(U15-PB18A-Pad42) -> /PB18A
- U15 pad 43: unconnected-(U15-PB18B-Pad43) -> /PB18B
- U15 pad 45: unconnected-(U15-PB18C-Pad45) -> /PB18C
- U15 pad 47: unconnected-(U15-PB18D-Pad47) -> /PB18D
- U15 pad 48: unconnected-(U15-PB20C/SN-Pad48) -> /lcmxo2-cpld-block/CPLD_SPI_CS
- U15 pad 49: unconnected-(U15-PB20D/SI/SISPI-Pad49) -> /lcmxo2-cpld-block/CPLD_MOSI
- U15 pad 50: GND -> Net-(D10-K)
- U15 pad 53: unconnected-(U15-PR9D-Pad53) -> /CPLD_B7_PR9D
- U15 pad 54: unconnected-(U15-PR9C-Pad54) -> /CPLD_B6_PR9C
- U15 pad 57: unconnected-(U15-PR9B-Pad57) -> /CPLD_B5_PR9B
- U15 pad 58: unconnected-(U15-PR9A-Pad58) -> /CPLD_B4_PR9A
- U15 pad 62: unconnected-(U15-PR5D/PCLKC1_0-Pad62) -> /lcmxo2-cpld-block/PR5D/PCLKC1_0
- U15 pad 63: unconnected-(U15-PR5C/PCLKT1_0-Pad63) -> /lcmxo2-cpld-block/PR5C/PCLKT1_0
- U15 pad 64: unconnected-(U15-PR5B-Pad64) -> /lcmxo2-cpld-block/PR5B
- U15 pad 65: unconnected-(U15-PR5A-Pad65) -> /lcmxo2-cpld-block/PR5A
- U15 pad 66: unconnected-(U15-PR4D-Pad66) -> /lcmxo2-cpld-block/PR4D
- U15 pad 67: unconnected-(U15-PR4C-Pad67) -> /lcmxo2-cpld-block/PR4C
- U15 pad 68: unconnected-(U15-PR4B-Pad68) -> /lcmxo2-cpld-block/PR4B
- U15 pad 69: unconnected-(U15-PR4A-Pad69) -> /lcmxo2-cpld-block/PR4A
- U15 pad 70: unconnected-(U15-PR3B-Pad70) -> /lcmxo2-cpld-block/PR3B
- U15 pad 71: unconnected-(U15-PR3A-Pad71) -> /lcmxo2-cpld-block/PR3A
- U15 pad 74: unconnected-(U15-PR2B-Pad74) -> /lcmxo2-cpld-block/PR2B
- U15 pad 75: unconnected-(U15-PR2A-Pad75) -> /lcmxo2-cpld-block/PR2A
- U15 pad 78: unconnected-(U15-PT16C-Pad78) -> /lcmxo2-cpld-block/PT16C
- U15 pad 83: unconnected-(U15-PT15B-Pad83) -> /lcmxo2-cpld-block/PT15B
- U15 pad 84: unconnected-(U15-PT15A-Pad84) -> /lcmxo2-cpld-block/PT15A
- U15 pad 85: /lcmxo2-cpld-block/PT12D/SDA/PCLKC0_0 -> /lcmxo2-cpld-block/CPLD_SDA
- U15 pad 86: /lcmxo2-cpld-block/PT12C/SCL/PCLKT0_0 -> /lcmxo2-cpld-block/CPLD_SCL
- U15 pad 87: unconnected-(U15-PT12B/PCLKC0_1-Pad87) -> /lcmxo2-cpld-block/PT12B/PCLKC0_1
- U15 pad 88: unconnected-(U15-PT12A/PCLKT0_1-Pad88) -> /lcmxo2-cpld-block/PT12A/PCLKT0_1
- U15 pad 96: unconnected-(U15-PT10B-Pad96) -> /CPLD_B1_PT10B
- U15 pad 97: unconnected-(U15-PT10A-Pad97) -> /CPLD_B0_PT10A
- U15 pad 98: unconnected-(U15-PT9B-Pad98) -> /CPLD_B3_PT9B
- U15 pad 99: unconnected-(U15-PT9A-Pad99) -> /CPLD_B2_PT9A
- U5 pad 10: unconnected-(U5-MDAT--Pad10) -> Net-(U5-MDAT-)
- U5 pad 11: unconnected-(U5-MDAT+-Pad11) -> Net-(U5-MDAT+)
- U5 pad 12: unconnected-(U5-MCLKIN−-Pad12) -> Net-(U5-MCLKIN−)
- U5 pad 13: unconnected-(U5-MCLKIN+-Pad13) -> Net-(U5-MCLKIN+)
- U5 pad 2: unconnected-(U5-VIN+-Pad2) -> Net-(U5-VIN+)
- U5 pad 3: unconnected-(U5-VIN--Pad3) -> Net-(U5-VIN-)
- U6 pad 25: /ice40-for-gpio/IOT_36b -> /IOT_36b
- U6 pad 26: /ice40-for-gpio/IOT_39a -> /IOT_39a
- U6 pad 27: /ice40-for-gpio/IOT_38b -> /IOT_38b
- U6 pad 32: /ice40-for-gpio/IOT_43a -> /IOT_43a
- U6 pad 34: /ice40-for-gpio/IOT_44b -> /IOT_44b
- U6 pad 35: /ice40-for-gpio/IOT_46b_G0 -> /ICE_CLOCK
- U6 pad 36: /ice40-for-gpio/IOT_48b -> /IOT_48b
- U6 pad 37: /ice40-for-gpio/IOT_45a_G1 -> /IOT_45a_G1

Commit message: update the  source code
Parts:
- removed J20: Conn_02x04_Top_Bottom, Connector_PinHeader_2.54mm:PinHeader_2x04_P2.54mm_Vertical
- added J22: RPI-TO-CPLD, Connector_PinHeader_2.54mm:PinHeader_2x05_P2.54mm_Vertical, F.Cu at (144.9, 108.0)
- added J23: CPLD-TO-RPI, Connector_PinHeader_2.54mm:PinHeader_2x05_P2.54mm_Vertical, F.Cu at (139.8, 88.9)
- added J24: CPLD-TO-RPI, Connector_PinHeader_2.54mm:PinHeader_2x05_P2.54mm_Vertical, F.Cu at (198.2, 72.4)
- J21: value Conn_02x04_Top_Bottom -> Conn_02x05_Top_Bottom; footprint Connector_PinHeader_2.54mm:PinHeader_2x04_P2.54mm_Vertical -> Connector_PinHeader_2.54mm:PinHeader_2x05_P2.54mm_Vertical
Connections:
- net /lcmxo2-cpld-block/CPLDK_SCK renamed /CPLDK_SCK
- net /lcmxo2-cpld-block/CPLD_MISO renamed /CPLD_MISO
- net /lcmxo2-cpld-block/CPLD_MOSI renamed /CPLD_MOSI
- net /lcmxo2-cpld-block/CPLD_SCL renamed /CPLD_SCL
- net /lcmxo2-cpld-block/CPLD_SDA renamed /CPLD_SDA
- net /lcmxo2-cpld-block/CPLD_SPI_CS renamed /CPLD_SPI_CS
- net /lcmxo2-cpld-block/CPLD_SPI_MCS renamed /CPLD_SPI_MCS
- A1 pad 21: /ICE_CDONE -> /GPIO16_SPI0_RX
- A1 pad 22: /CPLD_B0_PT10A -> /GPIO17_SPI0_CSn
- A1 pad 24: /CPLD_B1_PT10B -> /GPIO18_SPI0_SCK
- A1 pad 25: /CPLD_B2_PT9A -> /GPIO19_SPI0_TX
- A1 pad 26: /CPLD_B3_PT9B -> /GPIO20_I2C0_SDA
- A1 pad 27: /CPLD_B4_PR9A -> /GPIO21_I2C0_SCL
- A1 pad 29: /CPLD_B5_PR9B -> /ICE_CDONE
- A1 pad 31: unconnected-(A1-GPIO26_ADC0-Pad31) -> /GPIO26_ADC0
- A1 pad 32: /CPLD_B6_PR9C -> /GPIO27_ADC1
- A1 pad 34: /CPLD_B7_PR9D -> unconnected-(A1-GPIO28_ADC2-Pad34)
- J21 pad 1: /CPLD_B0_PT10A -> unconnected-(J21-Pin_1-Pad1)
- J21 pad 2: /CPLD_B1_PT10B -> unconnected-(J21-Pin_2-Pad2)
- J21 pad 3: /CPLD_B2_PT9A -> unconnected-(J21-Pin_3-Pad3)
- J21 pad 4: /CPLD_B3_PT9B -> unconnected-(J21-Pin_4-Pad4)
- J21 pad 5: /CPLD_B7_PR9D -> unconnected-(J21-Pin_5-Pad5)
- J21 pad 6: /CPLD_B6_PR9C -> unconnected-(J21-Pin_6-Pad6)
- J21 pad 7: /CPLD_B5_PR9B -> unconnected-(J21-Pin_7-Pad7)
- J21 pad 8: /CPLD_B4_PR9A -> unconnected-(J21-Pin_8-Pad8)
- U15 pad 12: unconnected-(U15-PL5A/PCLKT3_1-Pad12) -> /CPLD_CLOCK

Commit message: update the  source code
Parts:
- removed C11, C12: 100n, Capacitor_SMD:C_0402_1005Metric
- removed C34: 4.7u, Capacitor_SMD:C_0603_1608Metric
- removed J10: Jumpber, Connector_PinHeader_1.27mm:PinHeader_1x03_P1.27mm_Vertical
- removed J11, J9: Jumper, Connector_PinHeader_1.27mm:PinHeader_1x03_P1.27mm_Vertical
- removed J21: Conn_02x05_Top_Bottom, Connector_PinHeader_2.54mm:PinHeader_2x05_P2.54mm_Vertical
- removed J6, J7, J8: Conn_01x12, Connector_PinHeader_1.27mm:PinHeader_1x12_P1.27mm_Vertical
- removed Q1, Q2, Q3, Q4: 2N7002K, Package_TO_SOT_SMD:SOT-23
- removed R11, R12, R14, R17, R18: 1.2K, Resistor_SMD:R_0402_1005Metric
- removed R40, R41, R44, R45, R48: 10k, Resistor_SMD:R_0402_1005Metric
- removed R42, R43, R46, R47: 330R, Resistor_SMD:R_0402_1005Metric
- removed R8: 1R, Resistor_SMD:R_0402_1005Metric
- removed TP1: TestPoint, Connector_Pin:Pin_D0.7mm_L6.5mm_W1.8mm_FlatFork
- removed U10: LTC-3743KD, KiCadLocal:LTC-3743KD
- removed U3: LMV321, Package_TO_SOT_SMD:SOT-23-5
- removed U9: 74HC595D, PCM_JLCPCB:SOIC-16_3.9x9.9mm_P1.27mm
- added J20: Conn_01x10, Connector_PinHeader_2.54mm:PinHeader_1x10_P2.54mm_Vertical, F.Cu at (143.6, 96.6)
- added JP1: Jumper, Connector_PinHeader_2.54mm:PinHeader_1x03_P2.54mm_Vertical, F.Cu at (142.3, 73.3)
- added JP2: Jumper, Connector_PinHeader_2.54mm:PinHeader_1x03_P2.54mm_Vertical, F.Cu at (146.1, 73.3)
- added JP3: Jumper, Connector_PinHeader_2.54mm:PinHeader_1x03_P2.54mm_Vertical, F.Cu at (149.9, 73.3)
- added JP4: Jumper, Connector_PinHeader_2.54mm:PinHeader_1x03_P2.54mm_Vertical, F.Cu at (157.5, 73.3)
- added JP5: Jumper, Connector_PinHeader_2.54mm:PinHeader_1x03_P2.54mm_Vertical, F.Cu at (165.1, 73.3)
- added JP6: Jumper, Connector_PinHeader_2.54mm:PinHeader_1x03_P2.54mm_Vertical, F.Cu at (161.3, 73.3)
- J2: value Conn_01x02 -> TO-LCD; footprint TerminalBlock_Phoenix:TerminalBlock_Phoenix_PT-1,5-2-3.5-H_1x02_P3.50mm_Horizontal -> KiCadLocal:CON_536470274_MOL
- J22, J23, J24: footprint Connector_PinHeader_2.54mm:PinHeader_2x05_P2.54mm_Vertical -> Connector_PinHeader_2.54mm:PinHeader_2x06_P2.54mm_Vertical
- moved SW4 80.7 mm to (209.9, 45.8), turned to 180 degrees
- moved SW3 75.5 mm to (209.6, 41.3), turned to 180 degrees
- moved J22 73.5 mm to (132.2, 35.6), turned to 90 degrees
- moved J23 44.4 mm to (162.7, 127.0)
- moved J2 44.1 mm to (144.1, 88.4), turned to 180 degrees
- moved R29 24.6 mm to (168.8, 73.4), turned to 90 degrees
- moved C18 23.3 mm to (172.1, 73.6), turned to -90 degrees
- moved R28 19.8 mm to (170.2, 77.5), turned to -90 degrees
- moved C17 19.2 mm to (168.8, 77.6), turned to 90 degrees
- moved R31 18.3 mm to (167.7, 73.5), turned to -90 degrees
- moved C19 17.9 mm to (167.7, 77.6), turned to 90 degrees
- moved R30 17.7 mm to (183.7, 78.4), turned to -90 degrees
- moved D5 16.2 mm to (123.3, 38.9)
- moved J15 7.88 mm to (133.4, 96.6), turned to 0 degrees
- moved J5 5.12 mm to (162.7, 35.6)
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Connections:
- net /displays/MATRIX_SPI_MOSI renamed /MATRIX_SPI_MOSI
- net /displays/MATRIX_SPI_SCK renamed /MATRIX_SPI_SCK
- net /displays/MATRIX_SPI_nCS renamed /MATRIX_SPI_nCS
- J2 pad 1: Net-(J2-Pin_1) -> /DIG_1
- J2 pad 2: Net-(J2-Pin_2) -> /DIG_2
- J22 pad 10: +3.3V -> /GPIO27_ADC1
- J22 pad 5: GND -> /ICE_CLOCK
- J22 pad 6: /GPIO20_I2C0_SDA -> GND
- J22 pad 7: /GPIO21_I2C0_SCL -> /GPIO20_I2C0_SDA
- J22 pad 8: /GPIO26_ADC0 -> /GPIO21_I2C0_SCL
- J22 pad 9: /GPIO27_ADC1 -> /GPIO26_ADC0
- J23 pad 1: /GPIO18_SPI0_SCK -> /CPLDK_SCK
- J23 pad 10: +3.3V -> /CPLD_CLOCK
- J23 pad 2: /GPIO19_SPI0_TX -> /CPLD_MOSI
- J23 pad 3: /GPIO16_SPI0_RX -> /CPLD_MISO
- J23 pad 4: /GPIO17_SPI0_CSn -> /CPLD_SPI_CS
- J23 pad 5: GND -> /CPLD_CLOCK
- J23 pad 6: /GPIO20_I2C0_SDA -> GND
- J23 pad 7: /GPIO21_I2C0_SCL -> /CPLD_SDA
- J23 pad 8: /GPIO26_ADC0 -> /CPLD_SCL
- J23 pad 9: /GPIO27_ADC1 -> /CPLD_SPI_MCS
- J24 pad 10: +3.3V -> /CPLD_B0_PT10A
- J24 pad 5: GND -> /CPLD_CLOCK
- J24 pad 6: /CPLD_B3_PT9B -> GND
- J24 pad 7: /CPLD_B2_PT9A -> /CPLD_B3_PT9B
- J24 pad 8: /CPLD_B1_PT10B -> /CPLD_B2_PT9A
- J24 pad 9: /CPLD_B0_PT10A -> /CPLD_B1_PT10B
- U15 pad 10: unconnected-(U15-PL4B-Pad10) -> /PL4B
- U15 pad 34: unconnected-(U15-PB9A/PCLKT2_0-Pad34) -> /PB9A/PCLKT2_0
- U15 pad 35: unconnected-(U15-PB9B/PCLKC2_0-Pad35) -> /PB9B/PCLKC2_0
- U15 pad 36: unconnected-(U15-PB11C-Pad36) -> /PB11C
- U15 pad 37: unconnected-(U15-PB11D-Pad37) -> /PB11D
- U15 pad 38: unconnected-(U15-PB11A/PCLKT2_1-Pad38) -> /PB11A/PCLKT2_1
- U15 pad 51: unconnected-(U15-PR10D-Pad51) -> /PR10D
- U15 pad 52: unconnected-(U15-PR10C-Pad52) -> /PR10C
- U15 pad 59: unconnected-(U15-PR8D-Pad59) -> /PR8D
- U15 pad 60: unconnected-(U15-PR8C-Pad60) -> /PR8C
- U15 pad 61: unconnected-(U15-PR8A-Pad61) -> /PR8A
- U15 pad 9: unconnected-(U15-PL4A-Pad9) -> /PL4A
