File: stm32-fpga-bootloader.kicad_pcb (KiCad board)
At the start: 2 copper layers, 100 x 100 mm, 175 parts, among them J12 LEDX, J13 LEDY, J14 USB_C_Receptacle_USB2.0_14P, J15 Conn_ST_STDC14, J16 PMOD, J17 Raspberry_Pi_2_3, J18 Conn_ST_STDC14, J19 Conn_01x02, J2 TO-LCD, J20 Conn_01x10, J22 RPI-TO-CPLD, J23 CPLD-TO-RPI, J24 CPLD-TO-RPI, J3 Conn_01x02, J4 USB_C_Receptacle_USB2.0_14P, J5 PMOD, Q5 2N7002K, Q6 2N7002K, Q7 2N7002K, SW2 RUN, SW3 ICE_BTN, SW4 ICE_RST, U11 MAX7221xNG, U12 93LCxxA, U13 AMS1117-3.3, U14 FT2232HQ, U15 LCMXO2-1200HC-4TG100I, U4 LMV321, U5 ACPL-798J-500E, U6 ICE40UP5K-SG48ITR, U7 W25Q128JVS, U8 LP5907MFX-1.2, Y2 12Mhz

Commit message: update the  source code
Parts:
- moved J2 50.5 mm to (193.4, 99.5)
- moved R31 26.0 mm to (193.1, 79.0)
- moved C19 25.7 mm to (193.1, 81.2), turned to -90 degrees
- moved D5 14.8 mm to (132.3, 50.7), turned to 0 degrees
- moved C20 11.5 mm to (128.5, 39.1)
- moved JP4 7.30 mm to (150.2, 72.6)
- moved JP5 7.30 mm to (157.8, 72.6)
- moved JP6 7.30 mm to (154.0, 72.6)
- moved JP1 7.14 mm to (135.1, 72.8)
- moved JP2 7.14 mm to (138.9, 72.8)
- moved JP3 7.14 mm to (142.7, 72.8)
- moved D1 5.51 mm to (210.5, 50.4)
- moved D2 5.51 mm to (210.5, 54.1)
- moved D3 5.51 mm to (210.4, 56.8)
- moved R15 5.51 mm to (207.5, 56.8)
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Routing:
- net /ENCODER_BTN: track 0.00 -> 42.1 mm
- net /ENCODER_A: track 0.00 -> 28.2 mm
- net /ENCODER_B: track 0.00 -> 18.2 mm

Commit message: Update the source code
Parts:
- removed C36, C38, C39: 10uF, Capacitor_SMD:C_0603_1608Metric
- removed C37, C42, C46, C47, C48, C49, C50, C51: 100n, Capacitor_SMD:C_0402_1005Metric
- removed C40, C41: 10pF, Capacitor_SMD:C_0402_1005Metric
- removed C43, C44: 4.7u, Capacitor_SMD:C_0603_1608Metric
- removed C45: 1uF, Capacitor_SMD:C_0603_1608Metric
- removed D9: D_Schottky, Diode_SMD:D_SOD-123
- removed FB1, FB2: 600R@100Mhz, Inductor_SMD:L_0603_1608Metric
- removed J14, J4: USB_C_Receptacle_USB2.0_14P, Connector_USB:USB_C_Receptacle_G-Switch_GT-USB-7010ASV
- removed J15: Conn_ST_STDC14, Connector_PinHeader_1.27mm:PinHeader_2x07_P1.27mm_Vertical
- removed J20: Conn_01x10, Connector_PinHeader_2.54mm:PinHeader_1x10_P2.54mm_Vertical
- removed R56, R57, R58: 10k, Resistor_SMD:R_0402_1005Metric
- removed R59, R60, R69: 2.2k, Resistor_SMD:R_0402_1005Metric
- removed R61: 12k@1%, Resistor_SMD:R_0402_1005Metric
- removed R62, R63, R64, R65: 0R, Resistor_SMD:R_0402_1005Metric
- removed R66, R67, R68: 5.1k, Resistor_SMD:R_0402_1005Metric
- removed U12: 93LCxxA, Package_SO:SOIC-8_3.9x4.9mm_P1.27mm
- removed U13: AMS1117-3.3, Package_TO_SOT_SMD:SOT-223-3_TabPin2
- removed U14: FT2232HQ, Package_DFN_QFN:QFN-64-1EP_9x9mm_P0.5mm_EP4.35x4.35mm
- removed Y2: 12Mhz, Crystal:Crystal_SMD_3225-4Pin_3.2x2.5mm
- added A2: RaspberryPi_Pico, Module:RaspberryPi_Pico_Common_THT, F.Cu at (115.6, 92.3)
- moved U5 63.0 mm to (132.1, 108.8)
- moved C16 55.2 mm to (252.9, 115.2)
- moved D11 55.2 mm to (241.1, 131.2)
- moved J19 55.2 mm to (248.0, 134.2)
- moved R72 55.2 mm to (237.6, 130.9)
- moved R73 55.2 mm to (237.6, 115.0)
- moved R74 55.2 mm to (237.6, 117.0)
- moved R75 55.2 mm to (237.6, 119.0)
- moved R76 55.2 mm to (237.6, 121.0)
- moved R77 55.2 mm to (237.6, 123.0)
- moved R78 55.2 mm to (237.6, 125.0)
- moved R79 55.2 mm to (237.6, 132.9)
- moved R80 55.2 mm to (237.6, 134.9)
- moved R81 55.2 mm to (237.6, 136.9)
- moved R82 55.2 mm to (241.0, 115.3)
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Connections:
- net /D+ renamed Net-(J4-Pin_2)
- R25 pad 2: /ICE_X2 -> /IOB_20a
- R26 pad 1: /D- -> Net-(J4-Pin_1)
- U6 pad 10: /IOB_18a -> /ICE_USB_P
- U6 pad 9: /IOB_16a -> /ICE_USB_N

Commit message: Update the source files
Parts:
- removed C52, C53, C54, C55, C56, C57, C58, C59, C60, C61: 100n, Capacitor_SMD:C_0402_1005Metric
- removed FB5, FB6: 600R@100Mhz, Inductor_SMD:L_0603_1608Metric
- removed J16: PMOD, Connector_PinSocket_2.54mm:PinSocket_2x06_P2.54mm_Horizontal
- removed J17: Raspberry_Pi_2_3, Connector_PinHeader_2.54mm:PinHeader_2x20_P2.54mm_Vertical
- removed J18: Conn_ST_STDC14, Connector_PinHeader_1.27mm:PinHeader_2x07_P1.27mm_Vertical
- removed J19: Conn_01x02, TerminalBlock_Phoenix:TerminalBlock_Phoenix_PT-1,5-2-3.5-H_1x02_P3.50mm_Horizontal
- removed J22: RPI-TO-CPLD, Connector_PinHeader_2.54mm:PinHeader_2x06_P2.54mm_Vertical
- removed J23, J24: CPLD-TO-RPI, Connector_PinHeader_2.54mm:PinHeader_2x06_P2.54mm_Vertical
- removed Q5, Q6, Q7: 2N7002K, Package_TO_SOT_SMD:SOT-23
- removed R70, R71: 2.2k, Resistor_SMD:R_0402_1005Metric
- removed R72, R79, R80, R81, R87: 10k, Resistor_SMD:R_0402_1005Metric
- removed R73, R74, R75, R76, R77, R78: 100R, Resistor_SMD:R_0402_1005Metric
- removed R82, R83, R84, R85, R86: 1.2K, Resistor_SMD:R_0603_1608Metric
- removed U11: MAX7221xNG, Package_DIP:DIP-24_W7.62mm
- removed U15: LCMXO2-1200HC-4TG100I, Package_QFP:TQFP-100_14x14mm_P0.5mm
- added C1: 10uF, Capacitor_SMD:C_0603_1608Metric, F.Cu at (141.3, 105.6)
- added C10: 4.7u, Capacitor_SMD:C_0603_1608Metric, F.Cu at (134.5, 113.4)
- added C11: 100n, Capacitor_SMD:C_0402_1005Metric, F.Cu at (275.3, 21.8)
- added C12: 100n, Capacitor_SMD:C_0402_1005Metric, F.Cu at (275.3, 23.7)
- added C2: 100n, Capacitor_SMD:C_0402_1005Metric, F.Cu at (118.5, 120.2)
- added C3: 10uF, Capacitor_SMD:C_0603_1608Metric, F.Cu at (144.7, 105.5)
- added C34: 100n, Capacitor_SMD:C_0402_1005Metric, F.Cu at (187.7, 99.3)
- added C36: 100n, Capacitor_SMD:C_0402_1005Metric, F.Cu at (181.2, 99.4)
- added C37: 100n, Capacitor_SMD:C_0402_1005Metric, F.Cu at (177.3, 99.5)
- added C38: 100n, Capacitor_SMD:C_0402_1005Metric, F.Cu at (177.7, 119.5)
- added C39: 100n, Capacitor_SMD:C_0402_1005Metric, F.Cu at (173.6, 114.5)
- added C4: 10uF, Capacitor_SMD:C_0603_1608Metric, F.Cu at (141.2, 116.5)
- added C40: 100n, Capacitor_SMD:C_0402_1005Metric, F.Cu at (187.7, 119.6)
- added C41: 100n, Capacitor_SMD:C_0402_1005Metric, F.Cu at (173.6, 105.5)
- added C42: 100n, Capacitor_SMD:C_0402_1005Metric, F.Cu at (173.5, 108.6)
- added C43: 100n, Capacitor_SMD:C_0402_1005Metric, F.Cu at (189.7, 119.4)
- added C44: 100n, Capacitor_SMD:C_0402_1005Metric, F.Cu at (130.5, 105.4)
- added C45: 100n, Capacitor_SMD:C_0402_1005Metric, F.Cu at (126.9, 105.2)
- added C46: 100n, Capacitor_SMD:C_0402_1005Metric, F.Cu at (127.9, 105.2)
- added C5: 10pF, Capacitor_SMD:C_0402_1005Metric, F.Cu at (136.3, 113.0)
- added C6: 10pF, Capacitor_SMD:C_0402_1005Metric, F.Cu at (136.4, 107.6)
- added C7: 4.7u, Capacitor_SMD:C_0603_1608Metric, F.Cu at (136.7, 116.8)
- added C8: 100n, Capacitor_SMD:C_0402_1005Metric, F.Cu at (134.9, 116.2)
- added C9: 100n, Capacitor_SMD:C_0402_1005Metric, F.Cu at (126.4, 115.5)
- added D9: RED, LED_SMD:LED_0603_1608Metric, F.Cu at (191.6, 97.7)
- added FB1: 600R@100Mhz, Inductor_SMD:L_0603_1608Metric, F.Cu at (194.4, 114.7)
- added FB2: 600R@100Mhz, Inductor_SMD:L_0603_1608Metric, F.Cu at (189.0, 98.7)
- added J1: USB_C_Receptacle_USB2.0_14P, Connector_USB:USB_C_Receptacle_G-Switch_GT-USB-7010ASV, F.Cu at (116.4, 109.9)
- added J10: LEDX, Connector_PinSocket_2.54mm:PinSocket_1x08_P2.54mm_Vertical, F.Cu at (173.6, 35.9)
- added J11: LEDY, Connector_PinSocket_2.54mm:PinSocket_1x08_P2.54mm_Vertical, F.Cu at (173.6, 63.8)
- added J14: CPLD_JTAG, Connector_PinHeader_2.54mm:PinHeader_1x06_P2.54mm_Vertical, F.Cu at (161.6, 104.8)
- added J6: Conn_01x02, TerminalBlock_Phoenix:TerminalBlock_Phoenix_PT-1,5-2-3.5-H_1x02_P3.50mm_Horizontal, F.Cu at (208.5, 74.4)
- added J7: TO-LCD, KiCadLocal:CON_536470274_MOL, F.Cu at (206.6, 104.5)
- added J8: USB_C_Receptacle_USB2.0_14P, Connector_USB:USB_C_Receptacle_G-Switch_GT-USB-7010ASV, F.Cu at (117.0, 70.9)
- added Q1: 2N7002K, Package_TO_SOT_SMD:SOT-23, F.Cu at (187.7, 46.0)
- added Q2: 2N7002K, Package_TO_SOT_SMD:SOT-23, F.Cu at (187.8, 50.0)
- added Q3: 2N7002K, Package_TO_SOT_SMD:SOT-23, F.Cu at (187.7, 54.0)
- added R1: 27R, Resistor_SMD:R_0402_1005Metric, F.Cu at (123.4, 108.8)
- added R11: 1.2K, Resistor_SMD:R_0402_1005Metric, F.Cu at (208.1, 60.9)
- added R12: 10k, Resistor_SMD:R_0402_1005Metric, F.Cu at (134.5, 105.7)
- added R14: 1.2K, Resistor_SMD:R_0402_1005Metric, F.Cu at (272.9, 35.2)
- added R17: 1.2K, Resistor_SMD:R_0402_1005Metric, F.Cu at (272.9, 37.2)
- added R18: 1.2K, Resistor_SMD:R_0402_1005Metric, F.Cu at (272.9, 39.2)
- added R2: 27R, Resistor_SMD:R_0402_1005Metric, F.Cu at (123.5, 110.0)
- added R3: 10k, Resistor_SMD:R_0402_1005Metric, F.Cu at (130.2, 120.7)
- added R4: 1k, Resistor_SMD:R_0402_1005Metric, F.Cu at (134.8, 109.1)
- added R40: 1.2K, Resistor_SMD:R_0402_1005Metric, F.Cu at (139.6, 46.8)
- added R41: 1.2K, Resistor_SMD:R_0402_1005Metric, F.Cu at (138.6, 46.8)
- added R42: 10k, Resistor_SMD:R_0402_1005Metric, F.Cu at (121.7, 48.8)
- added R43: 10k, Resistor_SMD:R_0402_1005Metric, F.Cu at (122.3, 57.8)
- added R44: 10k, Resistor_SMD:R_0402_1005Metric, F.Cu at (121.8, 56.3)
- added R45: 100R, Resistor_SMD:R_0402_1005Metric, F.Cu at (145.3, 51.0)
- added R46: 10k, Resistor_SMD:R_0402_1005Metric, F.Cu at (185.2, 46.8)
- added R47: 10k, Resistor_SMD:R_0402_1005Metric, F.Cu at (185.3, 50.8)
- added R48: 10k, Resistor_SMD:R_0402_1005Metric, F.Cu at (185.2, 54.7)
- added R5: 1.2K, Resistor_SMD:R_0402_1005Metric, F.Cu at (123.6, 114.2)
- added R56: 2.2k, Resistor_SMD:R_0402_1005Metric, F.Cu at (185.5, 98.7)
- added R57: 2.2k, Resistor_SMD:R_0402_1005Metric, F.Cu at (185.5, 97.7)
- added R58: 10k, Resistor_SMD:R_0402_1005Metric, F.Cu at (191.8, 100.2)
- added R59: 0R, Resistor_SMD:R_0603_1608Metric, F.Cu at (157.1, 107.2)
- added R6: 1.2K, Resistor_SMD:R_0402_1005Metric, F.Cu at (119.2, 102.6)
- added R60: 0R, Resistor_SMD:R_0603_1608Metric, F.Cu at (157.1, 104.6)
- added R61: 0R, Resistor_SMD:R_0603_1608Metric, F.Cu at (157.1, 109.8)
- added R62: 0R, Resistor_SMD:R_0603_1608Metric, F.Cu at (157.1, 112.6)
- added R8: 1.2K, Resistor_SMD:R_0402_1005Metric, F.Cu at (208.1, 58.3)
- added SW1: BOOT, EasyEDA_Lib:SW-SMD_L3.9-W3.0-P4.45, F.Cu at (130.6, 126.7)
- added SW5: BOOT, EasyEDA_Lib:SW-SMD_L3.9-W3.0-P4.45, F.Cu at (125.2, 126.5)
- added U1: AMS1117-3.3, Package_TO_SOT_SMD:SOT-223-3_TabPin2, F.Cu at (143.3, 111.0)
- added U10: RP2040, Package_DFN_QFN:QFN-56-1EP_7x7mm_P0.4mm_EP3.2x3.2mm, F.Cu at (129.5, 110.6)
- added U2: W25Q128JVS, Package_SO:SOIC-8_5.3x5.3mm_P1.27mm, F.Cu at (123.8, 118.9)
- added U3: LMV321, Package_TO_SOT_SMD:SOT-23-5, F.Cu at (271.3, 23.2)
- added U9: LCMXO2-1200HC-4TG100I, Package_QFP:TQFP-100_14x14mm_P0.5mm, F.Cu at (183.7, 109.5)
- added Y1: 12Mhz, Crystal:Crystal_SMD_3225-4Pin_3.2x2.5mm, F.Cu at (137.2, 110.3)
- C13, C14: value 100n -> 10n
- C18, C19: value 10n -> 4.7u; footprint Capacitor_SMD:C_0402_1005Metric -> Capacitor_SMD:C_0603_1608Metric
- C20, C21, C24, C27, C28, C35: value 4.7u -> 100n; footprint Capacitor_SMD:C_0603_1608Metric -> Capacitor_SMD:C_0402_1005Metric
- C22, C25, C26, C29, C30: value 100n -> 4.7u; footprint Capacitor_SMD:C_0402_1005Metric -> Capacitor_SMD:C_0603_1608Metric
- C31: value 4.7u -> 10uF
- C33: value 10uF -> 100n; footprint Capacitor_SMD:C_0603_1608Metric -> Capacitor_SMD:C_0402_1005Metric
- J12: value LEDX -> PMOD; footprint Connector_PinSocket_2.54mm:PinSocket_1x08_P2.54mm_Vertical -> Connector_PinSocket_2.54mm:PinSocket_2x06_P2.54mm_Horizontal
- J13: value LEDY -> Raspberry_Pi_2_3; footprint Connector_PinSocket_2.54mm:PinSocket_1x08_P2.54mm_Vertical -> Connector_PinHeader_2.54mm:PinHeader_2x20_P2.54mm_Vertical
- J2: value TO-LCD -> Conn_01x02; footprint KiCadLocal:CON_536470274_MOL -> TerminalBlock_Phoenix:TerminalBlock_Phoenix_PT-1,5-2-3.5-H_1x02_P3.50mm_Horizontal
- J3: value Conn_01x02 -> RPI-TO-CPLD; footprint TerminalBlock_Phoenix:TerminalBlock_Phoenix_PT-1,5-2-3.5-H_1x02_P3.50mm_Horizontal -> Connector_PinHeader_2.54mm:PinHeader_2x06_P2.54mm_Vertical
- R10: value 10k -> 10R
- R13: value 10R -> 1R
- R19: value 1R -> 10k
- R20: value 1.2K -> 1.5K
- R21, R22: value 1.2K -> 27R
- R23, R24: footprint Resistor_SMD:R_0402_1005Metric -> Resistor_SMD:R_0603_1608Metric
- R25: value 1.5K -> 1.2K; footprint Resistor_SMD:R_0402_1005Metric -> Resistor_SMD:R_0603_1608Metric
- R26, R27: value 27R -> 1.2K; footprint Resistor_SMD:R_0402_1005Metric -> Resistor_SMD:R_0603_1608Metric
- R30: value PEC11S-9213K-S0015 -> 100R; footprint EasyEDA_Lib:RES-ADJ-SMD_PEC11S-9213K-S0015 -> Resistor_SMD:R_0603_1608Metric
- R31, R36: value 10k -> 100R; footprint Resistor_SMD:R_0402_1005Metric -> Resistor_SMD:R_0603_1608Metric
- R32: value 10k -> PEC11S-9213K-S0015; footprint Resistor_SMD:R_0402_1005Metric -> EasyEDA_Lib:RES-ADJ-SMD_PEC11S-9213K-S0015
- R33, R34, R35: value 1.2K -> 100R; footprint Resistor_SMD:R_0402_1005Metric -> Resistor_SMD:R_0603_1608Metric
- R39: value 100R -> 1.2K
- R52: value 10k -> 9.53k
- R55: value 9.53k -> 10k
- R9: value 1.2K -> 10k
- U4: value LMV321 -> ACPL-798J-500E; footprint Package_TO_SOT_SMD:SOT-23-5 -> EasyEDA_Lib:SO-16_L10.3-W7.5-P1.27-LS10.6-BL; moved to B.Cu
- U5: value ACPL-798J-500E -> ICE40UP5K-SG48ITR; footprint EasyEDA_Lib:SO-16_L10.3-W7.5-P1.27-LS10.6-BL -> Package_DFN_QFN:QFN-48-1EP_7x7mm_P0.5mm_EP5.6x5.6mm
- U6: value ICE40UP5K-SG48ITR -> W25Q128JVS; footprint Package_DFN_QFN:QFN-48-1EP_7x7mm_P0.5mm_EP5.6x5.6mm -> Package_SO:SOIC-8_5.3x5.3mm_P1.27mm
- U7: value W25Q128JVS -> LP5907MFX-1.2; footprint Package_SO:SOIC-8_5.3x5.3mm_P1.27mm -> Package_TO_SOT_SMD:SOT-23-5
- U8: value LP5907MFX-1.2 -> MAX7221xNG; footprint Package_TO_SOT_SMD:SOT-23-5 -> Package_DIP:DIP-24_W7.62mm
- moved R13 146.6 mm to (283.4, 31.5), turned to -90 degrees
- moved C15 130.1 mm to (252.0, 85.5)
- moved D11 128.4 mm to (115.9, 102.6)
- moved D4 110.5 mm to (115.8, 116.8), turned to 0 degrees
- moved J2 97.2 mm to (290.2, 30.0)
- moved J12 96.7 mm to (136.3, 125.1)
- moved R19 94.0 mm to (205.8, 45.3), turned to 90 degrees
- moved R15 90.2 mm to (286.8, 13.8)
- moved R16 90.2 mm to (286.8, 16.4)
- moved R27 84.4 mm to (207.3, 81.7)
- moved R26 84.4 mm to (207.3, 80.0), turned to 180 degrees
- moved R9 83.0 mm to (125.9, 38.6), turned to 180 degrees
- moved R36 81.6 mm to (200.4, 86.9), turned to 0 degrees
- moved U4 78.3 mm to (205.7, 83.2), turned to -90 degrees
- moved R23 78.3 mm to (203.0, 74.4), turned to 180 degrees
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Connections:
- A2 pad 1: unconnected-(A2-GPIO0-Pad1) -> /CPLD_B0_PT10A
- A2 pad 10: unconnected-(A2-GPIO7-Pad10) -> /CPLD_B7_PR9D
- A2 pad 14: unconnected-(A2-GPIO10-Pad14) -> /CPLDK_SCK
- A2 pad 2: unconnected-(A2-GPIO1-Pad2) -> /CPLD_B1_PT10B
- A2 pad 21: unconnected-(A2-GPIO16-Pad21) -> /CPLD_MISO
- A2 pad 22: unconnected-(A2-GPIO17-Pad22) -> /CPLD_SPI_CS
- A2 pad 24: unconnected-(A2-GPIO18-Pad24) -> /CPLDK_SCK
- A2 pad 25: unconnected-(A2-GPIO19-Pad25) -> /CPLD_MOSI
- A2 pad 26: unconnected-(A2-GPIO20-Pad26) -> /CPLD_SDA
- A2 pad 27: unconnected-(A2-GPIO21-Pad27) -> /CPLD_SCL
- A2 pad 29: unconnected-(A2-GPIO22-Pad29) -> /CPLD_SPI_MCS
- A2 pad 4: unconnected-(A2-GPIO2-Pad4) -> /CPLD_B2_PT9A
- A2 pad 5: unconnected-(A2-GPIO3-Pad5) -> /CPLD_B3_PT9B
- A2 pad 6: unconnected-(A2-GPIO4-Pad6) -> /CPLD_B4_PR9A
- A2 pad 7: unconnected-(A2-GPIO5-Pad7) -> /CPLD_B5_PR9B
- A2 pad 9: unconnected-(A2-GPIO6-Pad9) -> /CPLD_B6_PR9C
- C13 pad 1: +3.3V -> /ENCODER_A
- C14 pad 1: /ADC0 -> /ENCODER_B
- C17 pad 1: /ENCODER_A -> /ENCODER_BTN
- C18 pad 1: /ENCODER_B -> +3.3V
- C19 pad 1: /ENCODER_BTN -> +3.3V
- C24 pad 1: +3.3V -> GND
- C24 pad 2: GND -> +3.3V
- C26 pad 1: GND -> VBUS
- C26 pad 2: +3.3V -> GND
- C28 pad 1: VBUS -> Net-(U5D-VCCPLL)
- C29 pad 1: +3.3V -> Net-(U5D-VCCPLL)
- C30 pad 1: Net-(U6D-VCCPLL) -> +1V2
- C31 pad 1: Net-(U6D-VCCPLL) -> Net-(D8-K)
- C32 pad 1: +1V2 -> +5V
- C33 pad 1: Net-(D8-K) -> /lcmxo2-cpld-block/VCCIO1
- C35 pad 1: +5V -> /lcmxo2-cpld-block/VCCIO1
- D10 pad 1: Net-(D10-K) -> /lcmxo2-cpld-block/VCC
- D10 pad 2: Net-(D10-A) -> /lcmxo2-cpld-block/VCCIO0
- D11 pad 2: /lcmxo2-cpld-block/PT17D/DONE -> Net-(D11-A)
- D4 pad 2: /ICE_CDONE -> Net-(D4-A)
- FB3 pad 2: Net-(C52-Pad1) -> /lcmxo2-cpld-block/VCCIO2
- FB4 pad 2: Net-(D10-A) -> /lcmxo2-cpld-block/VCCIO3
- J12 pad 1: Net-(J12-Pin_1) -> /lcmxo2-cpld-block/PL8A
- J12 pad 2: Net-(J12-Pin_2) -> /lcmxo2-cpld-block/PL8B
- J12 pad 3: Net-(J12-Pin_3) -> /lcmxo2-cpld-block/PL5D
- J12 pad 4: Net-(J12-Pin_4) -> /lcmxo2-cpld-block/PL8D
- J12 pad 5: Net-(J12-Pin_5) -> /lcmxo2-cpld-block/PL5C
- J12 pad 6: Net-(J12-Pin_6) -> /lcmxo2-cpld-block/PL8C
- J12 pad 7: Net-(J12-Pin_7) -> /lcmxo2-cpld-block/PL9B/PCLKC3_0
- J12 pad 8: Net-(J12-Pin_8) -> /lcmxo2-cpld-block/PL9A/PCLKT3_0
- J13 pad 1: Net-(J13-Pin_1) -> unconnected-(J13-3V3-Pad1)_1
- J13 pad 2: Net-(J13-Pin_2) -> unconnected-(J13-5V-Pad2)_1
- J13 pad 3: Net-(J13-Pin_3) -> /CPLD_SDA
- J13 pad 4: Net-(J13-Pin_4) -> unconnected-(J13-5V-Pad2)
- J13 pad 5: Net-(J13-Pin_5) -> /CPLD_SCL
- J13 pad 6: Net-(J13-Pin_6) -> GND
- J13 pad 7: Net-(J13-Pin_7) -> /lcmxo2-cpld-block/PT15B
- J13 pad 8: Net-(J13-Pin_8) -> /lcmxo2-cpld-block/PB6A
- J2 pad 1: /DIG_1 -> Net-(J2-Pin_1)
- J2 pad 2: /DIG_2 -> Net-(J2-Pin_2)
- J3 pad 1: Net-(J3-Pin_1) -> /GPIO18_SPI0_SCK
- J3 pad 2: Net-(J3-Pin_2) -> /GPIO19_SPI0_TX
- JP1 pad 1: /IOT_48b -> /IOT_44b
- JP1 pad 2: /MATRIX_SPI_SCK -> /MATRIX_SPI_nCS
- JP1 pad 3: /PR10D -> /PR10C
- JP2 pad 1: /IOT_39a -> /IOT_38b
- JP2 pad 2: /MATRIX_SPI_MOSI -> /ENCODER_A
- JP2 pad 3: /PR8D -> /PB15A
- JP3 pad 1: /IOT_44b -> /IOT_39a
- JP3 pad 2: /MATRIX_SPI_nCS -> /MATRIX_SPI_MOSI
- JP3 pad 3: /PR10C -> /PR8D
- JP4 pad 1: /IOT_38b -> /IOT_36b
- JP4 pad 2: /ENCODER_A -> /ENCODER_B
- JP4 pad 3: /PB15A -> /PB15B
- JP5 pad 1: /IOT_36b -> /IOT_48b
- JP5 pad 2: /ENCODER_B -> /MATRIX_SPI_SCK
- JP5 pad 3: /PB15B -> /PR10D
- R10 pad 1: +3.3V -> Net-(A1-GPIO10)
- R10 pad 2: Net-(A1-RUN) -> /ICE_CLOCK
- R13 pad 1: Net-(A1-GPIO10) -> Net-(J2-Pin_1)
- R13 pad 2: /ICE_CLOCK -> Net-(J2-Pin_2)
- R15 pad 1: /LED2 -> Net-(J2-Pin_2)
- R15 pad 2: Net-(D3-A) -> Net-(U3--)
- R16 pad 1: +3.3V -> Net-(U3-+)
- R16 pad 2: /ICE_CDONE -> GND
- R19 pad 1: Net-(J3-Pin_1) -> +3.3V
- R19 pad 2: Net-(J3-Pin_2) -> /ICE_BTN
- R20 pad 1: Net-(J3-Pin_1) -> /D+
- R20 pad 2: Net-(U4-+) -> /IOB_20a
- R21 pad 1: Net-(J3-Pin_2) -> /D-
- R21 pad 2: Net-(U4--) -> /ICE_USB_N
- R22 pad 1: Net-(U4-+) -> /D+
- R22 pad 2: GND -> /ICE_USB_P
- R23 pad 1: Net-(U4--) -> Net-(J6-Pin_1)
- R24 pad 2: /ADC0 -> Net-(R24-Pad2)
- R25 pad 1: Net-(J4-Pin_2) -> GND
- R25 pad 2: /IOB_20a -> Net-(R24-Pad2)
- R26 pad 1: Net-(J4-Pin_1) -> Net-(R24-Pad2)
- R26 pad 2: /ICE_USB_N -> Net-(U4-VIN+)
- R27 pad 1: Net-(J4-Pin_2) -> GND
- R27 pad 2: /ICE_USB_P -> Net-(U4-VIN-)
- R30 pad 1: unconnected-(R30-Pad1) -> Net-(U4-MCLKIN−)
- R30 pad 2: unconnected-(R30-Pad2) -> Net-(U4-MCLKIN+)
- R31 pad 1: +3.3V -> Net-(U4-MDAT-)
- R31 pad 2: /ENCODER_BTN -> Net-(U4-MDAT+)
- R32 pad 1: +3.3V -> unconnected-(R32-Pad1)
- R32 pad 2: /ICE_nRST -> unconnected-(R32-Pad2)
- R33 pad 1: +3.3V -> /PB18A
- R33 pad 2: /ICE_CDONE -> Net-(U4-MCLKIN+)
- R34 pad 1: /ice40-for-gpio/ICE_LED1 -> /PB18B
- R34 pad 2: Net-(D6-A) -> Net-(U4-MCLKIN−)
- R35 pad 1: /ice40-for-gpio/ICE_LED2 -> /PB18C
- R35 pad 2: Net-(D7-A) -> Net-(U4-MDAT+)
- R36 pad 1: +3.3V -> /PB18D
- R36 pad 2: /ice40-for-gpio/ICE_SPI_IO3 -> Net-(U4-MDAT-)
- R37 pad 2: /ice40-for-gpio/ICE_SPI_IO2 -> /ENCODER_BTN
- R38 pad 2: /ICE_SPI_SS -> /ICE_nRST
- R39 pad 1: Net-(U6D-VCCPLL) -> +3.3V
- R39 pad 2: +1V2 -> /ICE_CDONE
- R49 pad 1: +3.3V -> +5V
- R49 pad 2: /MATRIX_SPI_nCS -> Net-(Q1-D)
- R50 pad 1: +3.3V -> +5V
- R50 pad 2: /MATRIX_SPI_SCK -> Net-(Q2-D)
- R51 pad 1: +3.3V -> +5V
- R51 pad 2: /MATRIX_SPI_MOSI -> Net-(Q3-D)
- R52 pad 2: Net-(Q5-D) -> Net-(U8-ISET)
- R53 pad 1: +5V -> +3.3V
- R53 pad 2: Net-(Q6-D) -> /lcmxo2-cpld-block/PT17D/DONE
- R54 pad 1: +5V -> +3.3V
- R54 pad 2: Net-(Q7-D) -> /lcmxo2-cpld-block/PT15D/PROGRAMN
- R55 pad 1: +5V -> +3.3V
- R55 pad 2: Net-(U11-ISET) -> /lcmxo2-cpld-block/PT15C/JTAGENB
- R9 pad 1: /LED1 -> +3.3V
- R9 pad 2: Net-(D2-A) -> Net-(A1-RUN)
- U4 pad 1: Net-(U4-+) -> +3.3V
- U4 pad 2: GND -> Net-(U4-VIN+)
- U4 pad 3: Net-(U4--) -> Net-(U4-VIN-)
- U4 pad 4: Net-(R23-Pad2) -> GND
- U4 pad 5: +3.3V -> unconnected-(U4-NC-Pad5)
- U5 pad 10: Net-(U5-MDAT-) -> /ICE_USB_P
- U5 pad 11: Net-(U5-MDAT+) -> /IOB_20a
- U5 pad 12: Net-(U5-MCLKIN−) -> /IOB_22a
- U5 pad 13: Net-(U5-MCLKIN+) -> /RPI_ICE3
- U5 pad 14: +3.3V -> /ICE_SPI_MOSI
- U5 pad 15: unconnected-(U5-NC-Pad15) -> /ICE_SPI_SCK
- U5 pad 16: GND -> /ICE_SPI_SS
- U5 pad 2: Net-(U5-VIN+) -> /IOB_6a
- U5 pad 3: Net-(U5-VIN-) -> /RPI_ICE0
- U5 pad 4: GND -> /IOB_8a
- U5 pad 5: unconnected-(U5-NC-Pad5) -> +3.3V
- U5 pad 6: unconnected-(U5-NC-Pad6) -> /IOB_13b
- U5 pad 7: +3.3V -> /ICE_CDONE
- U5 pad 8: GND -> /ICE_nRST
- U5 pad 9: GND -> /ICE_USB_N
- U6 pad 1: +3.3V -> /ICE_SPI_SS
- U6 pad 2: /IOB_6a -> /ICE_SPI_MISO
- U6 pad 3: /RPI_ICE0 -> /ice40-for-gpio/ICE_SPI_IO2
- U6 pad 4: /IOB_8a -> GND
- U6 pad 5: +3.3V -> /ICE_SPI_MOSI
- U6 pad 6: /IOB_13b -> /ICE_SPI_SCK
- U6 pad 7: /ICE_CDONE -> /ice40-for-gpio/ICE_SPI_IO3
- U6 pad 8: /ICE_nRST -> +3.3V
- U7 pad 1: /ICE_SPI_SS -> VBUS
- U7 pad 2: /ICE_SPI_MISO -> GND
- U7 pad 3: /ice40-for-gpio/ICE_SPI_IO2 -> VBUS
- U7 pad 4: GND -> unconnected-(U7-NC-Pad4)
- U7 pad 5: /ICE_SPI_MOSI -> +1V2
- U8 pad 1: VBUS -> Net-(Q3-D)
- U8 pad 2: GND -> Net-(J11-Pin_1)
- U8 pad 3: VBUS -> Net-(J11-Pin_5)
- U8 pad 4: unconnected-(U8-NC-Pad4) -> GND
- U8 pad 5: +1V2 -> Net-(J11-Pin_7)
Routing:
- net /ENCODER_BTN: track 42.1 -> 0.00 mm
- net /ENCODER_A: track 28.2 -> 0.00 mm
- net /ENCODER_B: track 18.2 -> 0.00 mm
