File: stm32-fpga-bootloader.kicad_pcb (KiCad board)
At the start: 4 copper layers, 100 x 100 mm, 212 parts, among them J1 USB_C_Receptacle_USB2.0_14P, J10 LEDX, J1001 DATA, J1002 JTAG JUMP, J1003 JTAG-LOG, J1004 Conn_01x08, J11 LEDY, J12 PMOD, J13 Raspberry_Pi_2_3, J15 Conn_01x02, J3 RPI-TO-CPLD, J5 PMOD, J6 Conn_01x02, J7 TO-LCD, J8 USB_C_Receptacle_USB2.0_14P, J9 PMOD, Q1 2N7002K, Q2 2N7002K, Q3 2N7002K, Q4 2N7002K, Q5 2N7002K, Q6 2N7002K, Q7 2N7002K, SW1 BOOT, SW2 RUN, SW3 ICE_BTN, SW4 ICE_RST, SW5 BOOT, SW6 BTN, SW7 BTN, SW8 BTN, U1 AMS1117-3.3, U10 RP2040, U1001 XC6206PxxxMR, U11 74HC595D, U12 LTC-3743KD, U13 ACPL-798J-500E, U2 W25Q128JVS, U4 ACPL-798J-500E, U5 ICE40UP5K-SG48ITR, U6 W25Q128JVS, U7 LP5907MFX-1.2, U8 MAX7221xNG, U9 LCMXO2-1200HC-4TG100I, Y1 12Mhz

Commit message: Update the source code
Parts:
- added J1005: JTAG JUMP, Connector_PinSocket_2.54mm:PinSocket_2x05_P2.54mm_Vertical, F.Cu at (211.0, 109.4)
- added J1006: JTAG JUMP, Connector_PinSocket_2.54mm:PinSocket_2x05_P2.54mm_Vertical, F.Cu at (229.9, 104.8)
- A1, A2: footprint Module:RaspberryPi_Pico_Common_THT -> KiCadLocal:RaspberryPi_Pico_Common_THT
- U13, U4: moved to F.Cu
- moved C48 147.0 mm to (268.3, 120.3)
- moved C49 147.0 mm to (267.9, 121.8)
- moved J1001 147.0 mm to (272.3, 112.6)
- moved J15 147.0 mm to (255.7, 115.3)
- moved R73 147.0 mm to (256.2, 111.5)
- moved R75 147.0 mm to (259.6, 114.2)
- moved R76 147.0 mm to (262.1, 113.4)
- moved R77 147.0 mm to (259.5, 117.5)
- moved R78 147.0 mm to (265.6, 113.6)
- moved R79 147.0 mm to (265.6, 117.1)
- moved R80 147.0 mm to (268.1, 114.5)
- moved R81 147.0 mm to (268.1, 112.9)
- moved R82 147.0 mm to (268.1, 116.3)
- moved R83 147.0 mm to (268.1, 117.9)
- moved R74 147.0 mm to (259.4, 111.4)
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Connections:
- J1002 pad 1: /PT10C/TDO -> GND
- J1002 pad 10: GND -> /TDI
- J1002 pad 2: /TDI -> GND
- J1002 pad 3: /PT10D/TDI -> /PT11D/TMS
- J1002 pad 4: /TDO -> /TMS
- J1002 pad 7: /PT11D/TMS -> /PT10D/TDI
- J1002 pad 8: /TMS -> /TDO
- J1002 pad 9: GND -> /PT10C/TDO
- J1004 pad 1: unconnected-(J1004-Pin_1-Pad1) -> /IOT_50b
- J1004 pad 2: unconnected-(J1004-Pin_2-Pad2) -> /IOB_13b
- J1004 pad 3: unconnected-(J1004-Pin_3-Pad3) -> /IOT_37a
- J1004 pad 4: unconnected-(J1004-Pin_4-Pad4) -> /IOB_20a
- J1004 pad 5: unconnected-(J1004-Pin_5-Pad5) -> /IOB_22a
- J1004 pad 6: unconnected-(J1004-Pin_6-Pad6) -> /IOB_23b
- J1004 pad 7: unconnected-(J1004-Pin_7-Pad7) -> /IOT_43a
- J1004 pad 8: unconnected-(J1004-Pin_8-Pad8) -> GND
- J13 pad 11: unconnected-(J13-GPIO17-Pad11) -> /lcmxo2-cpld-block/PR10C
- J13 pad 12: unconnected-(J13-GPIO18/PWM0-Pad12) -> /lcmxo2-cpld-block/PL10C
- J13 pad 13: unconnected-(J13-GPIO27-Pad13) -> /lcmxo2-cpld-block/PB15A
- J13 pad 15: unconnected-(J13-GPIO22-Pad15) -> /lcmxo2-cpld-block/PB11C
- J13 pad 16: unconnected-(J13-GPIO23-Pad16) -> /lcmxo2-cpld-block/PB11D
- J13 pad 18: unconnected-(J13-GPIO24-Pad18) -> /lcmxo2-cpld-block/PL10D
- J13 pad 22: unconnected-(J13-GPIO25-Pad22) -> /lcmxo2-cpld-block/PB11B/PCLKC2_1
- J13 pad 28: unconnected-(J13-ID_SC/GPIO1-Pad28) -> /lcmxo2-cpld-block/PL4A
- J13 pad 29: unconnected-(J13-GCLK1/GPIO5-Pad29) -> /lcmxo2-cpld-block/PR5C/PCLKT1_0
- J13 pad 31: unconnected-(J13-GCLK2/GPIO6-Pad31) -> /lcmxo2-cpld-block/PR5D/PCLKC1_0
- J13 pad 32: unconnected-(J13-PWM0/GPIO12-Pad32) -> /lcmxo2-cpld-block/PB9B/PCLKC2_0
- J13 pad 33: /lcmxo2-cpld-block/PL3B/PCLKC3_2 -> /lcmxo2-cpld-block/PB11A/PCLKT2_1
- J13 pad 35: unconnected-(J13-GPIO19/MISO1-Pad35) -> /lcmxo2-cpld-block/PT12B/PCLKC0_1
- J13 pad 36: unconnected-(J13-GPIO16-Pad36) -> /lcmxo2-cpld-block/PR10D
- J13 pad 37: unconnected-(J13-GPIO26-Pad37) -> /lcmxo2-cpld-block/PB15B
- J13 pad 38: unconnected-(J13-GPIO20/MOSI1-Pad38) -> /lcmxo2-cpld-block/PT12A/PCLKT0_1
- J13 pad 40: unconnected-(J13-GPIO21/SCLK1-Pad40) -> /lcmxo2-cpld-block/PB9A/PCLKT2_0
- J13 pad 7: unconnected-(J13-GCLK0/GPIO4-Pad7) -> /lcmxo2-cpld-block/PL4B
- J7 pad 18: /PR9A -> /PR8D
- J7 pad 20: /PR9B -> /PR9A
- R33 pad 1: /PB18A -> /isolated-measurements/PB18A
- R34 pad 1: /PB18B -> /isolated-measurements/PB18B
- R35 pad 1: /PB18C -> /isolated-measurements/PB18C
- R36 pad 1: /PB18D -> /isolated-measurements/PB18D
- U9 pad 10: unconnected-(U9-PL4B-Pad10) -> /lcmxo2-cpld-block/PL4B
- U9 pad 24: unconnected-(U9-PL10C-Pad24) -> /lcmxo2-cpld-block/PL10C
- U9 pad 25: unconnected-(U9-PL10D-Pad25) -> /lcmxo2-cpld-block/PL10D
- U9 pad 34: unconnected-(U9-PB9A/PCLKT2_0-Pad34) -> /lcmxo2-cpld-block/PB9A/PCLKT2_0
- U9 pad 35: unconnected-(U9-PB9B/PCLKC2_0-Pad35) -> /lcmxo2-cpld-block/PB9B/PCLKC2_0
- U9 pad 36: unconnected-(U9-PB11C-Pad36) -> /lcmxo2-cpld-block/PB11C
- U9 pad 37: unconnected-(U9-PB11D-Pad37) -> /lcmxo2-cpld-block/PB11D
- U9 pad 38: unconnected-(U9-PB11A/PCLKT2_1-Pad38) -> /lcmxo2-cpld-block/PB11A/PCLKT2_1
- U9 pad 39: unconnected-(U9-PB11B/PCLKC2_1-Pad39) -> /lcmxo2-cpld-block/PB11B/PCLKC2_1
- U9 pad 40: unconnected-(U9-PB15A-Pad40) -> /lcmxo2-cpld-block/PB15A
- U9 pad 41: unconnected-(U9-PB15B-Pad41) -> /lcmxo2-cpld-block/PB15B
- U9 pad 51: unconnected-(U9-PR10D-Pad51) -> /lcmxo2-cpld-block/PR10D
- U9 pad 52: unconnected-(U9-PR10C-Pad52) -> /lcmxo2-cpld-block/PR10C
- U9 pad 59: unconnected-(U9-PR8D-Pad59) -> /PR8D
- U9 pad 62: unconnected-(U9-PR5D/PCLKC1_0-Pad62) -> /lcmxo2-cpld-block/PR5D/PCLKC1_0
- U9 pad 63: unconnected-(U9-PR5C/PCLKT1_0-Pad63) -> /lcmxo2-cpld-block/PR5C/PCLKT1_0
- U9 pad 9: unconnected-(U9-PL4A-Pad9) -> /lcmxo2-cpld-block/PL4A
Routing:
- net /CPLD_B0_PT10A: track 0.00 -> 77.6 mm, vias 0 -> 3
- net /CPLD_B1_PT10B: track 0.00 -> 75.7 mm, vias 0 -> 3
- net /CPLD_B3_PT9B: track 0.00 -> 71.4 mm, vias 0 -> 6
- net /CPLD_B2_PT9A: track 0.00 -> 67.6 mm, vias 0 -> 1
- net /CPLD_SPI_MCS: track 0.00 -> 65.3 mm, vias 0 -> 5
- net /CPLD_MOSI: track 25.0 -> 88.1 mm, vias 0 -> 3
- net /lcmxo2-cpld-block/PL8B: track 0.00 -> 59.6 mm, vias 0 -> 1
- net /CPLD_B4_PL2C/L_GPLLT_IN: track 0.00 -> 58.8 mm, vias 0 -> 1
- net /CPLD_B5_PL2D/L_GPLLC_IN: track 0.00 -> 56.5 mm, vias 0 -> 1
- net /lcmxo2-cpld-block/PL8D: track 0.00 -> 56.2 mm, vias 0 -> 2
- net /lcmxo2-cpld-block/PL8A: track 0.00 -> 53.7 mm, vias 0 -> 1
- net /CPLD_B7_PL3B/PCLKC3_2: track 0.00 -> 53.0 mm, vias 0 -> 2
- net /lcmxo2-cpld-block/PL8C: track 0.00 -> 52.9 mm, vias 0 -> 2
- net /lcmxo2-cpld-block/PL5D: track 0.00 -> 51.2 mm, vias 0 -> 1
- net /lcmxo2-cpld-block/PT15A: track 1.85 -> 52.9 mm, vias 0 -> 2
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Other:
- board size 100 x 100 mm -> 161.3 x 100 mm

Commit message: Update the source code
Parts:
- removed C15, C48: 100n, Capacitor_SMD:C_0402_1005Metric
- removed C16, C49: 10uF, Capacitor_SMD:C_0603_1608Metric
- removed J1001: DATA, Connector_PinSocket_2.54mm:PinSocket_1x04_P2.54mm_Vertical
- removed J15: Conn_01x02, Connector_PinSocket_2.54mm:PinSocket_1x02_P2.54mm_Vertical
- removed J6: Conn_01x02, TerminalBlock_Phoenix:TerminalBlock_Phoenix_PT-1,5-2-3.5-H_1x02_P3.50mm_Horizontal
- removed R23, R24, R25, R26, R27, R73, R74, R75, R76, R77: 1.2K, Resistor_SMD:R_0603_1608Metric
- removed R30, R31, R33, R34, R35, R36, R78, R79, R80, R81, R82, R83: 100R, Resistor_SMD:R_0603_1608Metric
- removed U13, U4: ACPL-798J-500E, EasyEDA_Lib:SO-16_L10.3-W7.5-P1.27-LS10.6-BL
- J1006: value JTAG JUMP -> JTAG-LOG; footprint Connector_PinSocket_2.54mm:PinSocket_2x05_P2.54mm_Vertical -> Connector_PinSocket_2.54mm:PinSocket_1x03_P2.54mm_Vertical
- moved J1006 79.3 mm to (151.6, 92.7), turned to 90 degrees
- moved TP1 17.4 mm to (136.8, 75.8)
- moved C33 0.91 mm to (200.4, 112.3)
- moved FB1 0.88 mm to (200.9, 113.5)
- moved C39 0.49 mm to (178.4, 113.0)
Connections:
- J1005 pad 1: unconnected-(J1005-Pin_1-Pad1) -> /PB18C
- J1005 pad 2: unconnected-(J1005-Pin_2-Pad2) -> /PB18A
- J1005 pad 3: unconnected-(J1005-Pin_3-Pad3) -> /PB18D
- J1005 pad 4: unconnected-(J1005-Pin_4-Pad4) -> /PB18B
- J1006 pad 1: unconnected-(J1006-Pin_1-Pad1) -> /jtag-prog/SWD
- J1006 pad 2: unconnected-(J1006-Pin_2-Pad2) -> /jtag-prog/SWCLK
- J1006 pad 3: unconnected-(J1006-Pin_3-Pad3) -> GND
Routing:
- net /PR3A: track 0.00 -> 75.7 mm, vias 0 -> 3
- net /PR2B: track 0.00 -> 67.7 mm, vias 0 -> 1
- net /PR3B: track 0.00 -> 66.1 mm, vias 0 -> 3
- net /PR2A: track 0.00 -> 65.3 mm, vias 0 -> 2
- net /PR4A: track 0.00 -> 63.0 mm, vias 0 -> 3
- net /PR4B: track 0.00 -> 62.6 mm, vias 0 -> 3
- net /PR9D: track 0.00 -> 41.2 mm
- net /PR9C: track 0.00 -> 39.0 mm
- net /lcmxo2-cpld-block/PR10C: track 0.00 -> 38.2 mm, vias 0 -> 2
- net /lcmxo2-cpld-block/PL4B: track 0.00 -> 38.1 mm, vias 0 -> 2
- net /lcmxo2-cpld-block/PR5C/PCLKT1_0: track 0.00 -> 36.7 mm, vias 0 -> 1
- net /displays/SHIFT_REG_DATA: track 0.00 -> 33.3 mm, vias 0 -> 1
- net /displays/SHIFT_REG_OE: track 11.2 -> 44.0 mm
- net /displays/SHIFT_REG_nMCLR: track 0.00 -> 32.6 mm, vias 0 -> 1
- net /lcmxo2-cpld-block/PT12B/PCLKC0_1: track 0.00 -> 32.4 mm, vias 0 -> 1
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Other:
- board size 161.3 x 100 mm -> 100 x 100 mm
