File: displays.kicad_sch (KiCad schematic)
At the start: 31 parts, among them J3 LEDX, J4 LEDY, Q1 2N7002K, Q2 2N7002K, Q3 2N7002K, Q4 2N7002K, Q6 2N7002K, Q7 2N7002K, Q8 2N7002K, U11 74HC595D, U12 LTC-3743KD, U15 MAX7221xNG

Commit message: Update the design files
Parts:
- TP1: footprint Connector_Pin:Pin_D0.9mm_L10.0mm_W2.4mm_FlatFork -> Connector_Pin:Pin_D0.7mm_L6.5mm_W1.8mm_FlatFork
Connections:
- net SHIFT_REG_OE: now reaches R47.1, U11.13 (OE#)
Changed lines of the file:
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@@
+	)
+	(junction
+		(at 44.45 62.23)
+		(diameter 0)
+		(color 0 0 0 0)
 	)
 	(junction
@@
 		(pts
 			(xy 240.03 57.15) (xy 251.46 57.15)
+		)
+		(stroke
+			(width 0)
+			(type default)
+		)
+	)
+	(wire
+		(pts
+			(xy 40.64 62.23) (xy 44.45 62.23)
 		)
 		(stroke
@@
 		(shape input)
 		(at 194.31 107.95 180)
+		(effects
+			(font
+				(size 1.27 1.27)
+			)
+			(justify right)
+		)
+	)
+	(hierarchical_label "SHIFT_REG_OE"
+		(shape input)
+		(at 40.64 62.23 180)
 		(effects
 			(font
@@
 			)
 		)
-		(property "Footprint" "Connector_Pin:Pin_D0.9mm_L10.0mm_W2.4mm_FlatFork"
+		(property "Footprint" "Connector_Pin:Pin_D0.7mm_L6.5mm_W1.8mm_FlatFork"
 			(at 46.99 80.01 0)
 			(effects

Commit message: Update the schematic
Parts:
- U9: renamed from U11; footprint PCM_JLCPCB:SOIC-16_L9.9-W3.9-P1.27-LS6.0-BL -> PCM_JLCPCB:SOIC-16_3.9x9.9mm_P1.27mm
- renumbered C10 to C34, C14 to C35, J3 to J12, J4 to J13, Q4 to Q1, Q1 to Q4, Q8 to Q5, R47 to R40, R7 to R41, R58 to R42, R56 to R43, R9 to R44, R8 to R45, R57 to R46, R55 to R47, R11 to R48, R53 to R49, R49 to R50, R54 to R52, R50 to R53, R52 to R54, R46 to R55, U12 to U10, U15 to U11

Commit message: update the  source code
Parts:
- removed C34: 4.7u, Capacitor_SMD:C_0603_1608Metric, symbol Device:C_Small
- removed Q1, Q2, Q3, Q4: 2N7002K, Package_TO_SOT_SMD:SOT-23, symbol Transistor_FET:2N7002K
- removed R40, R41, R44, R45, R48: 10k, Resistor_SMD:R_0402_1005Metric, symbol Device:R_Small
- removed R42, R43, R46, R47: 330R, Resistor_SMD:R_0402_1005Metric, symbol Device:R_Small
- removed TP1: TestPoint, Connector_Pin:Pin_D0.7mm_L6.5mm_W1.8mm_FlatFork, symbol Connector:TestPoint
- removed U10: LTC-3743KD, KiCadLocal:LTC-3743KD, symbol KiCadLocal:LTC-3743KD
- removed U9: 74HC595D, PCM_JLCPCB:SOIC-16_3.9x9.9mm_P1.27mm, symbol PCM_JLCPCB-ICs:Shift Register, 1 In, 8 Out, 74HC595D,118
Connections:
- no-connect marks 14 -> 1

Commit message: Update the source code
Parts:
- renumbered C35 to C32, J12 to J10, J13 to J11, Q5 to Q1, Q6 to Q2, Q7 to Q3, R49 to R46, R50 to R47, R51 to R48, R52 to R49, R53 to R50, R54 to R51, R55 to R52, U11 to U8

Commit message: Update the source files
Parts:
- added J7: TO-LCD, KiCadLocal:CON_536470274_MOL, symbol Connector_Generic:Conn_02x11_Odd_Even
Connections:
- net +5V: now also J7.7 (Pin_7), J7.8 (Pin_8)
- net GND: now also J7.11 (Pin_11), J7.12 (Pin_12)
- new net CLOCK: J7.17 (Pin_17)
- new net DIG_1: J7.1 (Pin_1)
- new net DIG_2: J7.2 (Pin_2)
- new net DIG_3: J7.4 (Pin_4)
- new net DIG_4: J7.6 (Pin_6)
- new net DIG_DP: J7.3 (Pin_3)
- new net IO: J7.16 (Pin_16)
- new net KEY: J7.18 (Pin_18)
- new net LED_SEG: J7.15 (Pin_15)
- new net RTSW_A: J7.19 (Pin_19)
- new net RTSW_B: J7.20 (Pin_20)
- no-connect marks 1 -> 8

Commit message: Update the source files
Parts:
- added C47: 4.7u, Capacitor_SMD:C_0603_1608Metric, symbol Device:C_Small
- added J4001: Conn_01x08, Connector_PinSocket_2.54mm:PinSocket_1x08_P2.54mm_Vertical, symbol Connector_Generic:Conn_01x08
- added Q4, Q5, Q6, Q7: 2N7002K, Package_TO_SOT_SMD:SOT-23, symbol Transistor_FET:2N7002K
- added R63, R64, R67, R68, R70: 10k, Resistor_SMD:R_0402_1005Metric, symbol Device:R_Small
- added R65, R66, R69, R71: 330R, Resistor_SMD:R_0402_1005Metric, symbol Device:R_Small
- added TP1: TestPoint, TestPoint:TestPoint_Pad_1.0x1.0mm, symbol Connector:TestPoint
- added U11: 74HC595D, PCM_JLCPCB:SOIC-16_3.9x9.9mm_P1.27mm, symbol PCM_JLCPCB-ICs:Shift Register, 1 In, 8 Out, 74HC595D,118
- added U12: LTC-3743KD, KiCadLocal:LTC-3743KD, symbol KiCadLocal:LTC-3743KD
Connections:
- net +3.3V: now also C47.1, U11.16 (VCC)
- net GND: now also C47.2, Q4.2 (S), Q5.2 (S), Q6.2 (S), Q7.2 (S), R63.2, R64.2, R67.2, R68.2, R70.2, U11.8 (GND)
- new net: TP1.1, U11.9 (Q7S)
- new net: Q5.3 (D), R66.2
- new net: R65.1, U12.2 (D1)
- new net: Q4.3 (D), R65.2
- new net: R71.1, U12.10 (D4)
- new net: R69.1, U12.5 (D2)
- new net: R66.1, U12.8 (D3)
- new net: Q6.3 (D), R69.2
- new net: Q7.3 (D), R71.2
- new net 7SEG_A: U11.15 (Q0), U12.17 (A)
- new net 7SEG_B: U11.1 (Q1), U12.19 (B)
- new net 7SEG_C: U11.2 (Q2), U12.20 (C)
- new net 7SEG_D: U11.3 (Q3), U12.3 (D)
- new net 7SEG_D1: J4001.6 (Pin_6), Q4.1 (G), R64.1
- new net 7SEG_D2: J4001.7 (Pin_7), Q6.1 (G), R68.1
- new net 7SEG_D3: J4001.8 (Pin_8), Q5.1 (G), R67.1
- new net 7SEG_D4: Q7.1 (G), R70.1
- new net 7SEG_E: U11.4 (Q4), U12.11 (E), U12.21 (D1_E_AN)
- new net 7SEG_F: U11.5 (Q5), U12.18 (F)
- new net 7SEG_G: U11.6 (Q6), U12.22 (G)
- new net SHIFT_REG_CLK: J4001.4 (Pin_4), U11.11 (SHCP)
- new net SHIFT_REG_DATA: J4001.1 (Pin_1), U11.14 (DS)
- new net SHIFT_REG_OE: J4001.2 (Pin_2), R63.1, U11.13 (OE#)
- new net SHIFT_REG_STCLK: J4001.3 (Pin_3), U11.12 (STCP)
- new net SHIFT_REG_nMCLR: J4001.5 (Pin_5), U11.10 (MR#)
- no-connect marks 8 -> 21
Other:
- moved on the sheet: C32, J10, J11, J7, Q1, Q2, Q3, R46, R47, R48, R49, R50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

Commit message: Update the schematic
Parts:
- removed J4001: Conn_01x08, Connector_PinSocket_2.54mm:PinSocket_1x08_P2.54mm_Vertical, symbol Connector_Generic:Conn_01x08
- added J9: PMOD, Connector_PinSocket_2.54mm:PinSocket_2x06_P2.54mm_Vertical, symbol Connector_Generic:Conn_02x06_Odd_Even
- added R72: 10k, Resistor_SMD:R_0402_1005Metric, symbol Device:R_Small
- U11: footprint PCM_JLCPCB:SOIC-16_3.9x9.9mm_P1.27mm -> PCM_JLCPCB:SOIC-16_L9.9-W3.9-P1.27-LS6.0-BL
Connections:
- net +3.3V: now also J9.11 (Pin_11), J9.12 (Pin_12), R72.1
- net 7SEG_D1: now also J9.2 (Pin_2)
- net 7SEG_D2: now also J9.4 (Pin_4)
- net 7SEG_D3: now also J9.6 (Pin_6)
- net 7SEG_D4: now also J9.8 (Pin_8)
- net GND: now also J9.10 (Pin_10)
- net SHIFT_REG_CLK: now also J9.5 (Pin_5)
- net SHIFT_REG_DATA: now also J9.1 (Pin_1)
- net SHIFT_REG_OE: now also J9.9 (Pin_9)
- net SHIFT_REG_STCLK: now also J9.3 (Pin_3)
- net SHIFT_REG_nMCLR: now also J9.7 (Pin_7), R72.2
Other:
- note added: "TODO Update the pins orders in the Footprints"
- moved on the sheet: R63

Commit message: Update the schematic
Other:
- note removed: "TODO Update the pins orders in the Footprints"
Changed lines of the file:
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@@
-		)
-	)
-	(text "TODO\nUpdate the pins orders in the Footprints"
-		(exclude_from_sim no)
-		(at 88.9 169.672 0)
-		(effects
-			(font
-				(size 1.27 1.27)
-				(color 255 83 83 1)
-			)
 		)
 	)
