File: lcmxo2-cpld-block.kicad_sch (KiCad schematic)
At the start: 23 parts, among them J11 Raspberry_Pi_2_3, J12 Conn_ST_STDC14, J13 PMOD, U5 LCMXO2-1200HC-4TG100I, Y3 ASE-xxxMHz

Commit message: Update the schematic
Parts:
- removed C63: 100n, Capacitor_SMD:C_0402_1005Metric, symbol Device:C_Small
- removed Y3: ASE-xxxMHz, Oscillator:Oscillator_SMD_Abracon_ASE-4Pin_3.2x2.5mm_HandSoldering, symbol Oscillator:ASE-xxxMHz
- added D11: RED, LED_SMD:LED_0603_1608Metric, symbol Device:LED_Small
- added R72, R79, R80, R81: 10k, Resistor_SMD:R_0402_1005Metric, symbol Device:R_Small
- renumbered C61 to C52, C57 to C53, C62 to C54, C58 to C55, C59 to C56, C67 to C57, C66 to C58, C68 to C59, C65 to C60, C64 to C61, FB4 to FB3, FB3 to FB4, FB6 to FB5, FB5 to FB6, J13 to J16, J11 to J17, J12 to J18, R72 to R70, U5 to U15
Connections:
- net PL10C is gone; now on net UART_TX: U15.24 (PL10C)
- net PL9B/PCLKC3_0 is gone; now on net PL9B/PCLKC3_0: U15.21 (PL9B/PCLKC3_0)
- net PT12C/SCL/PCLKT0_0 is gone; now on net CPLD_SCL: R71.1, U15.86 (PT12C/SCL/PCLKT0_0)
- net PT12D/SDA/PCLKC0_0 is gone; now on net CPLD_SDA: R70.1, U15.85 (PT12D/SDA/PCLKC0_0)
- net +3.3V: now also R72.1, R79.1, R80.1, R81.1
- net GND: now also J17.14 (GND), J17.20 (GND), J17.25 (GND), J17.30 (GND), J17.34 (GND), J17.39 (GND), J17.6 (GND), J17.9 (GND), D11.1 (K); no longer U15.50 (VCC)
- net PL9A/PCLKT3_0: now also J16.8 (Pin_8)
- net PT15C/JTAGENB: now also R81.2
- net PT15D/PROGRAMN: now also R72.2
- net PT17C/INITN: now also R80.2
- net PT17D/DONE: now also D11.2 (A), R79.2
- net UART_RX: now also U15.25 (PL10D)
- net PL8A: now reaches J16.1 (Pin_1)
- net PL8A: now also U15.16 (PL8A)
- net PL8B: now reaches J16.2 (Pin_2)
- net PL8B: now also U15.17 (PL8B)
- net PL5D: now reaches J16.3 (Pin_3)
- net PL5D: now also U15.15 (PL5D)
- net PL8D: now reaches J16.4 (Pin_4)
- net PL8D: now also U15.19 (PL8D)
- net PL5C: now reaches J16.5 (Pin_5)
- net PL5C: now also U15.14 (PL5C)
- net PL8C: now reaches J16.6 (Pin_6)
- net PL8C: now also U15.18 (PL8C)
- net PL9B/PCLKC3_0: now reaches J16.7 (Pin_7)
- net PB6B: now reaches J17.10 (GPIO15/RXD)
- net PB6B: now also U15.30 (PB6B)
- net PR5D/PCLKC1_0: now reaches J17.11 (GPIO17)
- net PR5D/PCLKC1_0: now also U15.62 (PR5D/PCLKC1_0)
- net PR5C/PCLKT1_0: now reaches J17.12 (GPIO18/PWM0)
- net PR5C/PCLKT1_0: now also U15.63 (PR5C/PCLKT1_0)
- net PR2A: now reaches J17.13 (GPIO27)
- net PR2A: now also U15.75 (PR2A)
- net PR4B: now reaches J17.15 (GPIO22)
- net PR4B: now also U15.68 (PR4B)
- net PR4A: now reaches J17.16 (GPIO23)
- net PR4A: now also U15.69 (PR4A)
- net PR3B: now reaches J17.18 (GPIO24)
- net PR3B: now also U15.70 (PR3B)
- net CPLD_MOSI: now reaches J17.19 (MOSI0/GPIO10)
- net CPLD_MOSI: now also U15.49 (PB20D/SI/SISPI)
- net CPLD_MISO: now reaches J17.21 (MISO0/GPIO9)
- net CPLD_MISO: now also U15.32 (PB6D/SO/SPISO)
- net PR3A: now reaches J17.22 (GPIO25)
- net PR3A: now also U15.71 (PR3A)
- net CPLDK_SCK: now reaches J17.23 (SCLK0/GPIO11)
- net CPLDK_SCK: now also U15.31 (PB6C/MCLK/CCLK)
- net CPLD_SPI_CS: now reaches J17.24 (~{CE0}/GPIO8)
- net CPLD_SPI_CS: now also U15.48 (PB20C/SN)
- net CPLD_SPI_MCS: now reaches J17.26 (~{CE1}/GPIO7)
- net CPLD_SPI_MCS: now also U15.27 (PB4C/CSSPIN)
- net PB4D: now reaches J17.27 (ID_SD/GPIO0)
- net PB4D: now also U15.28 (PB4D)
- net PT16C: now reaches J17.28 (ID_SC/GPIO1)
- net PT16C: now also U15.78 (PT16C)
- net PT12A/PCLKT0_1: now reaches J17.29 (GCLK1/GPIO5)
- net PT12A/PCLKT0_1: now also U15.88 (PT12A/PCLKT0_1)
- net CPLD_SDA: now reaches J17.3 (SDA/GPIO2)
- net PT12B/PCLKC0_1: now reaches J17.31 (GCLK2/GPIO6)
- net PT12B/PCLKC0_1: now also U15.87 (PT12B/PCLKC0_1)
- net PT15A: now reaches J17.32 (PWM0/GPIO12)
- net PT15A: now also U15.84 (PT15A)
- net PL3B/PCLKC3_2: now reaches J17.33 (PWM1/GPIO13)
- net PL3B/PCLKC3_2: now also U15.4 (PL3B/PCLKC3_2)
- net PR5A: now reaches J17.35 (GPIO19/MISO1)
- net PR5A: now also U15.65 (PR5A)
- net PR5B: now reaches J17.36 (GPIO16)
- net PR5B: now also U15.64 (PR5B)
- net PR2B: now reaches J17.37 (GPIO26)
- net PR2B: now also U15.74 (PR2B)
- net PR4D: now reaches J17.38 (GPIO20/MOSI1)
- net PR4D: now also U15.66 (PR4D)
- net PR4C: now reaches J17.40 (GPIO21/SCLK1)
- net PR4C: now also U15.67 (PR4C)
- net CPLD_SCL: now reaches J17.5 (SCL/GPIO3)
- net PT15B: now reaches J17.7 (GCLK0/GPIO4)
- net PT15B: now also U15.83 (PT15B)
- net PB6A: now reaches J17.8 (GPIO14/TXD)
- net PB6A: now also U15.29 (PB6A)
- net at C56.2, D10.1 (K), U15.100 (VCC): now also U15.50 (VCC)
- net PL5B/PCLKC3_1: now reaches U15.13 (PL5B/PCLKC3_1)
- net PB15B: now reaches U15.41 (PB15B)
- net PB18A: now reaches U15.42 (PB18A)
- net PB18B: now reaches U15.43 (PB18B)
- net PB18C: now reaches U15.45 (PB18C)
- net PB18D: now reaches U15.47 (PB18D)
- no-connect marks 2 -> 5
Other:
- moved on the sheet: C52, C53, C54, C55, C56, C57, C58, C59, C60, C61, D10, FB3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

Commit message: Update the schematic
Connections:
- net PB11B/PCLKC2_1: now reaches U15.39 (PB11B/PCLKC2_1)
- net PB15A: now reaches U15.40 (PB15A)
- net CPLD_B7_PR9D: now reaches U15.53 (PR9D)
- net CPLD_B6_PR9C: now reaches U15.54 (PR9C)
- net CPLD_B5_PR9B: now reaches U15.57 (PR9B)
- net CPLD_B4_PR9A: now reaches U15.58 (PR9A)
- net CPLD_B1_PT10B: now reaches U15.96 (PT10B)
- net CPLD_B0_PT10A: now reaches U15.97 (PT10A)
- net CPLD_B3_PT9B: now reaches U15.98 (PT9B)
- net CPLD_B2_PT9A: now reaches U15.99 (PT9A)
Changed lines of the file:
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@@
+	(wire
+		(pts
+			(xy 82.55 100.33) (xy 91.44 100.33)
+		)
+		(stroke
+			(width 0)
+			(type default)
+		)
+	)
 	(wire
 		(pts
@@
 	(wire
 		(pts
+			(xy 163.83 158.75) (xy 157.48 158.75)
+		)
+		(stroke
+			(width 0)
+			(type default)
+		)
+	)
+	(wire
+		(pts
 			(xy 204.47 62.23) (xy 212.09 62.23)
 		)
@@
 	(wire
 		(pts
+			(xy 82.55 115.57) (xy 91.44 115.57)
+		)
+		(stroke
+			(width 0)
+			(type default)
+		)
+	)
+	(wire
+		(pts
 			(xy 104.14 30.48) (xy 114.3 30.48)
 		)
@@
 	(wire
 		(pts
+			(xy 82.55 118.11) (xy 91.44 118.11)
+		)
+		(stroke
+			(width 0)
+			(type default)
+		)
+	)
+	(wire
+		(pts
 			(xy 26.67 175.26) (xy 31.75 175.26)
 		)
@@
 	(wire
 		(pts
+			(xy 82.55 105.41) (xy 91.44 105.41)
+		)
+		(stroke
+			(width 0)
+			(type default)
+		)
+	)
+	(wire
+		(pts
 			(xy 72.39 163.83) (xy 91.44 163.83)
 		)
@@
 	(wire
 		(pts
+			(xy 82.55 102.87) (xy 91.44 102.87)
+		)
+		(stroke
+			(width 0)
+			(type default)
+		)
+	)
+	(wire
+		(pts
 			(xy 114.3 187.96) (xy 116.84 187.96)
 		)
@@
 	(wire
 		(pts
+			(xy 82.55 107.95) (xy 91.44 107.95)
+		)
+		(stroke
+			(width 0)
+			(type default)
+		)
+	)
+	(wire
+		(pts
 			(xy 13.97 172.72) (xy 31.75 172.72)
 		)
@@
 	(wire
 		(pts
+			(xy 163.83 156.21) (xy 157.48 156.21)
+		)
+		(stroke
+			(width 0)
+			(type default)
+		)
+	)
+	(wire
+		(pts
 			(xy 134.62 17.78) (xy 151.13 17.78)
 		)
@@
 	(wire
 		(pts
+			(xy 82.55 110.49) (xy 91.44 110.49)
+		)
+		(stroke
+			(width 0)
+			(type default)
+		)
+	)
+	(wire
+		(pts
 			(xy 121.92 187.96) (xy 127 187.96)
 		)
@@
 		(pts
 			(xy 163.83 153.67) (xy 157.48 153.67)
+		)
+		(stroke
+			(width 0)
+			(type default)
+		)
+	)
+	(wire
+		(pts
+			(xy 82.55 113.03) (xy 91.44 113.03)
 		)
 		(stroke
@@
 		)
 	)
+	(hierarchical_label "CPLD_B0_PT10A"
+		(shape passive)
+		(at 82.55 100.33 180)
+		(effects
+			(font
+				(size 1.27 1.27)
+			)
+			(justify right)
+		)
+	)
+	(hierarchical_label "CPLD_B4_PR9A"
+		(shape passive)
+		(at 82.55 110.49 180)
+		(effects
+			(font
+				(size 1.27 1.27)
+			)
+			(justify right)
+		)
+	)
 	(hierarchical_label "CPLD_SDA"
 		(shape passive)
@@
 		)
 	)
+	(hierarchical_label "CPLD_B6_PR9C"
+		(shape passive)
+		(at 82.55 115.57 180)
+		(effects
+			(font
+				(size 1.27 1.27)
+			)
+			(justify right)
+		)
+	)
 	(hierarchical_label "CPLD_SPI_MCS"
 		(shape passive)
@@
 		)
 	)
+	(hierarchical_label "CPLD_B5_PR9B"
+		(shape passive)
+		(at 82.55 113.03 180)
+		(effects
+			(font
+				(size 1.27 1.27)
+			)
+			(justify right)
+		)
+	)
 	(hierarchical_label "PT11D/TMS"
 		(shape passive)
@@
 		)
 	)
+	(hierarchical_label "CPLD_B1_PT10B"
+		(shape passive)
+		(at 82.55 102.87 180)
+		(effects
+			(font
+				(size 1.27 1.27)
+			)
+			(justify right)
+		)
+	)
 	(hierarchical_label "PT15D/PROGRAMN"
 		(shape passive)
@@
 		)
 	)
+	(hierarchical_label "CPLD_B3_PT9B"
+		(shape passive)
+		(at 82.55 107.95 180)
+		(effects
+			(font
+				(size 1.27 1.27)
+			)
+			(justify right)
+		)
+	)
+	(hierarchical_label "PB15A"
+		(shape passive)
+		(at 163.83 156.21 0)
+		(effects
+			(font
+				(size 1.27 1.27)
+			)
+			(justify left)
+		)
+	)
 	(hierarchical_label "CPLDK_SCK"
 		(shape passive)
@@
 		)
 	)
+	(hierarchical_label "CPLD_B2_PT9A"
+		(shape passive)
+		(at 82.55 105.41 180)
+		(effects
+			(font
+				(size 1.27 1.27)
+			)
+			(justify right)
+		)
+	)
 	(hierarchical_label "PT15C/JTAGENB"
 		(shape passive)
@@
 		)
 	)
+	(hierarchical_label "CPLD_B7_PR9D"
+		(shape passive)
+		(at 82.55 118.11 180)
+		(effects
+			(font
+				(size 1.27 1.27)
+			)
+			(justify right)
+		)
+	)
 	(hierarchical_label "CPLD_SCL"
 		(shape passive)
@@
 		(effects
 			(font
+				(size 1.27 1.27)
+			)
+			(justify left)
+		)
+	)
+	(hierarchical_label "PB11B/PCLKC2_1"
+		(shape passive)
+		(at 163.83 158.75 0)
+		(effects
+			(font

Commit message: update the  source code
Connections:
- net PL5A/PCLKT3_1: now reaches U15.12 (PL5A/PCLKT3_1)
Changed lines of the file:
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@@
+	(wire
+		(pts
+			(xy 176.53 115.57) (xy 157.48 115.57)
+		)
+		(stroke
+			(width 0)
+			(type default)
+		)
+	)
 	(wire
 		(pts
@@
 		)
 	)
+	(hierarchical_label "PL5A/PCLKT3_1"
+		(shape passive)
+		(at 176.53 115.57 0)
+		(effects
+			(font
+				(size 1.27 1.27)
+			)
+			(justify left)
+		)
+	)

Commit message: update the  source code
Connections:
- net PL4B: now reaches U15.10 (PL4B)
- net PB9A/PCLKT2_0: now reaches U15.34 (PB9A/PCLKT2_0)
- net PB9B/PCLKC2_0: now reaches U15.35 (PB9B/PCLKC2_0)
- net PB11C: now reaches U15.36 (PB11C)
- net PB11D: now reaches U15.37 (PB11D)
- net PB11A/PCLKT2_1: now reaches U15.38 (PB11A/PCLKT2_1)
- net PR10D: now reaches U15.51 (PR10D)
- net PR10C: now reaches U15.52 (PR10C)
- net PR8D: now reaches U15.59 (PR8D)
- net PR8C: now reaches U15.60 (PR8C)
- net PR8A: now reaches U15.61 (PR8A)
- net PL4A: now reaches U15.9 (PL4A)
Changed lines of the file:
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@@
+	(wire
+		(pts
+			(xy 160.02 161.29) (xy 157.48 161.29)
+		)
+		(stroke
+			(width 0)
+			(type default)
+		)
+	)
 	(wire
 		(pts
@@
 	(wire
 		(pts
-			(xy 162.56 173.99) (xy 157.48 173.99)
-		)
-		(stroke
-			(width 0)
-			(type default)
-		)
-	)
-	(wire
-		(pts
 			(xy 36.83 92.71) (xy 36.83 97.79)
 		)
@@
 	(wire
 		(pts
+			(xy 160.02 120.65) (xy 157.48 120.65)
+		)
+		(stroke
+			(width 0)
+			(type default)
+		)
+	)
+	(wire
+		(pts
 			(xy 267.97 147.32) (xy 270.51 147.32)
 		)
@@
 	(wire
 		(pts
+			(xy 160.02 168.91) (xy 157.48 168.91)
+		)
+		(stroke
+			(width 0)
+			(type default)
+		)
+	)
+	(wire
+		(pts
 			(xy 204.47 69.85) (xy 212.09 69.85)
 		)
@@
 	(wire
 		(pts
+			(xy 157.48 173.99) (xy 162.56 173.99)
+		)
+		(stroke
+			(width 0)
+			(type default)
+		)
+	)
+	(wire
+		(pts
 			(xy 270.51 146.05) (xy 270.51 147.32)
 		)
@@
 	(wire
 		(pts
+			(xy 160.02 166.37) (xy 157.48 166.37)
+		)
+		(stroke
+			(width 0)
+			(type default)
+		)
+	)
+	(wire
+		(pts
 			(xy 80.01 59.69) (xy 85.09 59.69)
 		)
@@
 	(wire
 		(pts
+			(xy 86.36 128.27) (xy 91.44 128.27)
+		)
+		(stroke
+			(width 0)
+			(type default)
+		)
+	)
+	(wire
+		(pts
 			(xy 134.62 186.69) (xy 134.62 187.96)
 		)
@@
 	(wire
 		(pts
+			(xy 160.02 118.11) (xy 157.48 118.11)
+		)
+		(stroke
+			(width 0)
+			(type default)
+		)
+	)
+	(wire
+		(pts
 			(xy 82.55 85.09) (xy 91.44 85.09)
 		)
@@
 	(wire
 		(pts
+			(xy 160.02 171.45) (xy 157.48 171.45)
+		)
+		(stroke
+			(width 0)
+			(type default)
+		)
+	)
+	(wire
+		(pts
 			(xy 29.21 170.18) (xy 31.75 170.18)
 		)
@@
 	(wire
 		(pts
+			(xy 86.36 123.19) (xy 91.44 123.19)
+		)
+		(stroke
+			(width 0)
+			(type default)
+		)
+	)
+	(wire
+		(pts
 			(xy 87.63 176.53) (xy 91.44 176.53)
 		)
@@
 	(wire
 		(pts
+			(xy 160.02 163.83) (xy 157.48 163.83)
+		)
+		(stroke
+			(width 0)
+			(type default)
+		)
+	)
+	(wire
+		(pts
 			(xy 163.83 153.67) (xy 157.48 153.67)
 		)
@@
 	(wire
 		(pts
+			(xy 86.36 130.81) (xy 91.44 130.81)
+		)
+		(stroke
+			(width 0)
+			(type default)
+		)
+	)
+	(wire
+		(pts
 			(xy 163.83 148.59) (xy 157.48 148.59)
 		)
@@
 	(wire
 		(pts
+			(xy 86.36 125.73) (xy 91.44 125.73)
+		)
+		(stroke
+			(width 0)
+			(type default)
+		)
+	)
+	(wire
+		(pts
 			(xy 160.02 30.48) (xy 151.13 30.48)
 		)
@@
 		(pts
 			(xy 132.08 186.69) (xy 132.08 187.96)
+		)
+		(stroke
+			(width 0)
+			(type default)
+		)
+	)
+	(wire
+		(pts
+			(xy 86.36 120.65) (xy 91.44 120.65)
 		)
 		(stroke
@@
 		)
 	)
+	(hierarchical_label "PB9B/PCLKC2_0"
+		(shape passive)
+		(at 160.02 168.91 0)
+		(effects
+			(font
+				(size 1.27 1.27)
+			)
+			(justify left)
+		)
+	)
 	(hierarchical_label "CPLD_B5_PR9B"
 		(shape passive)
@@
 		)
 	)
+	(hierarchical_label "PB9A/PCLKT2_0"
+		(shape passive)
+		(at 160.02 171.45 0)
+		(effects
+			(font
+				(size 1.27 1.27)
+			)
+			(justify left)
+		)
+	)
 	(hierarchical_label "PB18C"
 		(shape passive)
@@
 		)
 	)
+	(hierarchical_label "PL4B"
+		(shape passive)
+		(at 160.02 118.11 0)
+		(effects
+			(font
+				(size 1.27 1.27)
+			)
+			(justify left)
+		)
+	)
 	(hierarchical_label "PT15C/JTAGENB"
 		(shape passive)
@@
 		)
 	)
+	(hierarchical_label "PR8A"
+		(shape passive)
+		(at 86.36 125.73 180)
+		(effects
+			(font
+				(size 1.27 1.27)
+			)
+			(justify right)
+		)
+	)
 	(hierarchical_label "PT10C/TDO"
 		(shape passive)
@@
 		)
 	)
+	(hierarchical_label "PR10C"
+		(shape passive)
+		(at 86.36 123.19 180)
+		(effects
+			(font
+				(size 1.27 1.27)
+			)
+			(justify right)
+		)
+	)
 	(hierarchical_label "PT17D/DONE"
 		(shape passive)
@@
 		)
 	)
+	(hierarchical_label "PL4A"
+		(shape passive)
+		(at 160.02 120.65 0)
+		(effects
+			(font
+				(size 1.27 1.27)
+			)
+			(justify left)
+		)
+	)
 	(hierarchical_label "CPLD_B2_PT9A"
 		(shape passive)
@@
 		)
 	)
+	(hierarchical_label "PR8D"
+		(shape passive)
+		(at 86.36 128.27 180)
+		(effects
+			(font
+				(size 1.27 1.27)
+			)
+			(justify right)
+		)
+	)
 	(hierarchical_label "PT15C/JTAGENB"
 		(shape passive)
@@
 		)
 	)
+	(hierarchical_label "PB11A/PCLKT2_1"
+		(shape passive)
+		(at 160.02 161.29 0)
+		(effects
+			(font
+				(size 1.27 1.27)
+			)
+			(justify left)
+		)
+	)
 	(hierarchical_label "CPLD_SCL"
 		(shape passive)
@@
 		)
 	)
+	(hierarchical_label "PB11D"
+		(shape passive)
+		(at 160.02 163.83 0)
+		(effects
+			(font
+				(size 1.27 1.27)
+			)
+			(justify left)
+		)
+	)
 	(hierarchical_label "PB18B"
 		(shape passive)
@@
 		(effects
 			(font
+				(size 1.27 1.27)
+			)
+			(justify left)
+		)
+	)
+	(hierarchical_label "PR10D"
+		(shape passive)
+		(at 86.36 120.65 180)
+		(effects
+			(font
+				(size 1.27 1.27)
+			)
+			(justify right)
+		)
+	)
+	(hierarchical_label "PR8C"
+		(shape passive)
+		(at 86.36 130.81 180)
+		(effects
+			(font
+				(size 1.27 1.27)
+			)
+			(justify right)
+		)
+	)
+	(hierarchical_label "PB11C"
+		(shape passive)
+		(at 160.02 166.37 0)
+		(effects
+			(font

Commit message: Update the source code
Parts:
- added C43: 100n, Capacitor_SMD:C_0402_1005Metric, symbol Device:C_Small
- renumbered C52 to C33, C53 to C34, C54 to C35, C55 to C36, C56 to C37, C57 to C38, C58 to C39, C59 to C40, C60 to C41, C61 to C42, D11 to D9, FB3 to FB1, FB4 to FB2, FB5 to FB3, FB6 to FB4, J16 to J12, J17 to J13, J18 to J14, R79 to R53, R72 to R54, R81 to R55, R70 to R56, R71 to R57, R80 to R58, U15 to U9
Connections:
- net GND: now also C43.1
- net VCCIO3: now reaches C39.1, C41.1, C42.1, FB4.2, U9.11 (VCCIO3), U9.23 (VCCIO3), U9.5 (VCCIO3)
- net VCCIO1: now reaches C33.1, C35.1, FB1.2, U9.55 (VCCIO1), U9.73 (VCCIO1)
- net VCCIO2: now reaches C38.1, C40.1, FB3.2, U9.26 (VCCIO2), U9.46 (VCCIO2)
- net VCCIO0: now reaches C34.1, C36.1, D10.2 (A), FB2.2, U9.80 (VCCIO0), U9.93 (VCCIO0)
- net VCC: now reaches C37.2, D10.1 (K), U9.100 (VCC), U9.50 (VCC)
- net VCC: now also C43.2

Commit message: Update the source files
Parts:
- removed J14: Conn_ST_STDC14, Connector_PinHeader_1.27mm:PinHeader_2x07_P1.27mm_Vertical, symbol Connector:Conn_ST_STDC14
Connections:
- net UART_RX renamed PL10C
- net UART_TX renamed PL10D
- no-connect marks 5 -> 3
