File: isolated-measurements.kicad_sch (KiCad schematic)
At the start: 30 parts, among them J1001 DATA, J1006 JTAG JUMP, J14 Conn_01x02, J6 Conn_01x02, U13 ACPL-798J-500E, U4 ACPL-798J-500E

Commit message: Update the source code
Parts:
- removed C15, C48: 100n, Capacitor_SMD:C_0603_1608Metric, symbol Device:C_Small
- removed C16, C49: 10uF, Capacitor_SMD:C_0603_1608Metric, symbol Device:C_Small
- removed C52: 10n, Capacitor_SMD:C_0603_1608Metric, symbol Device:C_Small
- removed J1001: DATA, Connector_PinSocket_2.54mm:PinSocket_1x04_P2.54mm_Vertical, symbol Connector_Generic:Conn_01x04
- removed J1006: JTAG JUMP, Connector_PinSocket_2.54mm:PinSocket_2x05_P2.54mm_Vertical, symbol Connector_Generic:Conn_02x05_Odd_Even
- removed J14, J6: Conn_01x02, TerminalBlock_Phoenix:TerminalBlock_Phoenix_PT-1,5-2-3.5-H_1x02_P3.50mm_Horizontal, symbol Connector_Generic:Conn_01x02
- removed R23, R24, R25, R26, R27: 1.2K, Resistor_SMD:R_1206_3216Metric, symbol Device:R_Small
- removed R30, R31, R33, R34, R35, R36, R78, R79, R80, R81, R82, R83: 100R, Resistor_SMD:R_1206_3216Metric, symbol Device:R_Small
- removed R76, R77: 22R, Resistor_SMD:R_1206_3216Metric, symbol Device:R_Small
- removed U13, U4: ACPL-798J-500E, EasyEDA_Lib:SO-16_L10.3-W7.5-P1.27-LS10.6-BL, symbol KiCadLocal:ACPL-798J-500E
