File: jtag-prog.kicad_sch (KiCad schematic)
At the start: 32 parts, among them J1 USB_C_Receptacle_USB2.0_14P, SW1 BOOT, SW5 BOOT, U10 RP2040, U1001 XC6206PxxxMR, U2 W25Q128JVS, Y1 12Mhz

Commit message: Update the source code
Parts:
- added J1006: JTAG-LOG, Connector_PinSocket_2.54mm:PinSocket_1x03_P2.54mm_Vertical, symbol Connector_Generic:Conn_01x03
Connections:
- net GND: now also J1006.3 (Pin_3)
- net SWCLK: now also J1006.2 (Pin_2)
- net SWD: now also J1006.1 (Pin_1)
- no-connect marks 26 -> 22
Other:
- moved on the sheet: C5, C6, R4, Y1
